Commit message: feat: tool manipulator 구성 파일 및 초기 위치 추가; 제어 및 운동학 설정 업데이트

File: src/arm/tool_manipulator_moveit_config/config/tool_manipulator.urdf.xacro (robot description, xacro)
@@ -1,17 +1,9 @@
 <?xml version="1.0"?>
 <robot xmlns:xacro="http://www.ros.org/wiki/xacro" name="tool_manipulator">
-  <xacro:arg name="use_mock_hardware" default="true"/>
-  <xacro:arg name="use_mesh" default="true"/>
-  <xacro:include filename="$(find tool_manipulator_description)/urdf/tool_manipulator.urdf.xacro"/>
-  <!-- The CAD description has no hardware tag.  This self-contained mock
-       interface exists only for simulation and MoveIt integration. -->
-  <ros2_control name="ToolManipulatorMockSystem" type="system">
-    <hardware><plugin>mock_components/GenericSystem</plugin></hardware>
-    <joint name="base_joint"><command_interface name="position"/><state_interface name="position"><param name="initial_value">0</param></state_interface><state_interface name="velocity"/></joint>
-    <joint name="shoulder_joint"><command_interface name="position"/><state_interface name="position"><param name="initial_value">0</param></state_interface><state_interface name="velocity"/></joint>
-    <joint name="elbow_joint"><command_interface name="position"/><state_interface name="position"><param name="initial_value">0</param></state_interface><state_interface name="velocity"/></joint>
-    <joint name="wrist_pitch_joint"><command_interface name="position"/><state_interface name="position"><param name="initial_value">0</param></state_interface><state_interface name="velocity"/></joint>
-    <joint name="wrist_roll_joint"><command_interface name="position"/><state_interface name="position"><param name="initial_value">0</param></state_interface><state_interface name="velocity"/></joint>
-    <joint name="wrist_yaw_joint"><command_interface name="position"/><state_interface name="position"><param name="initial_value">0</param></state_interface><state_interface name="velocity"/></joint>
-  </ros2_control>
+    <xacro:arg name="initial_positions_file" default="initial_positions.yaml" />
+    <!-- Import tool_manipulator urdf file -->
+    <xacro:include filename="$(find tool_manipulator_description)/urdf/tool_manipulator.urdf.xacro" />
+    <!-- Import control_xacro -->
+    <xacro:include filename="tool_manipulator.ros2_control.xacro" />
+    <xacro:tool_manipulator_ros2_control name="FakeSystem" initial_positions_file="$(arg initial_positions_file)"/>
 </robot>
