Commit message: 왜안될가

File: src/arm/tool_manipulator_moveit_config/config/tool_manipulator.ros2_control.xacro (robot description, xacro)
@@ -41,5 +41,5 @@
     </ros2_control>
   </xacro:macro>
-  <xacro:macro name="dxl_joint" params="name spec wrap">
+  <xacro:macro name="dxl_joint" params="name spec state_wrap:=false command_nearest_turn:=false">
     <joint name="${name}">
       <xacro:if value="${spec['operating_mode'] == 1}">
@@ -59,5 +59,9 @@
       <param name="position_zero_offset">${spec['zero_raw'] * 2.0 * pi / 4096.0 - pi}</param>
       <param name="position_direction">${1.0 if spec['raw_increases_ccw'] else -1.0}</param>
-      <param name="position_wraparound">${wrap}</param>
+      <!-- Extended-position feedback may restart on another 2*pi branch.
+           Normalize only the ROS state; map position commands to the raw turn
+           nearest the measured motor position to avoid a full-revolution jump. -->
+      <param name="position_state_wraparound">${'true' if state_wrap else 'false'}</param>
+      <param name="position_command_nearest_turn">${'true' if command_nearest_turn else 'false'}</param>
     </joint>
   </xacro:macro>
@@ -119,8 +123,9 @@
           <param name="joint_to_transmission_matrix">1,0,0,0,0,1,0,0,0,0,1,0,0,0,0,1</param>
         </hardware>
-        <xacro:dxl_joint name="base_joint" spec="${j['base_joint']}" wrap="false"/>
-        <xacro:dxl_joint name="wrist_roll_joint" spec="${j['wrist_roll_joint']}" wrap="false"/>
-        <xacro:dxl_joint name="wrist_yaw_joint" spec="${j['wrist_yaw_joint']}" wrap="false"/>
-        <xacro:dxl_joint name="ee_joint" spec="${j['ee_joint']}" wrap="false"/>
+        <xacro:dxl_joint name="base_joint" spec="${j['base_joint']}"/>
+        <xacro:dxl_joint name="wrist_roll_joint" spec="${j['wrist_roll_joint']}"/>
+        <xacro:dxl_joint name="wrist_yaw_joint" spec="${j['wrist_yaw_joint']}"
+                         state_wrap="true" command_nearest_turn="true"/>
+        <xacro:dxl_joint name="ee_joint" spec="${j['ee_joint']}"/>
         <xacro:dxl_gpio name="base_motor" spec="${j['base_joint']}"/>
         <xacro:dxl_gpio name="wrist_roll_motor" spec="${j['wrist_roll_joint']}"/>
