Commit message: d

File: src/arm/tool_manipulator_description/urdf/tools/tool_2.xacro (robot description, xacro)
@@ -4,6 +4,6 @@
     <joint name="${prefix}tool_2_mount_joint" type="fixed"><parent link="${parent}"/><child link="${prefix}tool_2_link"/><origin xyz="0 0 0.012" rpy="${pi/2} 0 0"/></joint>
     <link name="${prefix}tool_2_link">
-      <visual><geometry><mesh filename="package://tool_manipulator_description/meshes/visual/long_drillbit.stl" scale="0.001 0.001 0.001"/></geometry><material name="motor_grey"/></visual>
-      <collision><geometry><mesh filename="package://tool_manipulator_description/meshes/collision/long_drillbit.stl" scale="0.001 0.001 0.001"/></geometry></collision>
+      <visual><geometry><mesh filename="package://tool_manipulator_description/meshes/visual/tool1_drill.stl" scale="0.001 0.001 0.001"/></geometry><material name="motor_grey"/></visual>
+      <collision><geometry><mesh filename="package://tool_manipulator_description/meshes/collision/tool1_drill.stl" scale="0.001 0.001 0.001"/></geometry></collision>
       <inertial><origin xyz="0 0.030 0"/><mass value="0.050"/><inertia ixx="0.00002" ixy="0" ixz="0" iyy="0.000004" iyz="0" izz="0.00002"/></inertial>
     </link>

Commit message: tool2 수정

File: src/arm/tool_manipulator_description/urdf/tools/tool_2.xacro (robot description, xacro)
@@ -2,5 +2,5 @@
 <robot xmlns:xacro="http://www.ros.org/wiki/xacro">
   <xacro:macro name="tool_2" params="prefix parent use_mesh:=false">
-    <joint name="${prefix}tool_2_mount_joint" type="fixed"><parent link="${parent}"/><child link="${prefix}tool_2_link"/><origin xyz="0 0 0.012" rpy="${pi/2} 0 0"/></joint>
+    <joint name="${prefix}tool_2_mount_joint" type="fixed"><parent link="${parent}"/><child link="${prefix}tool_2_link"/><origin xyz="0 0 0.012" rpy="0 0 0"/></joint>
     <link name="${prefix}tool_2_link">
       <visual><geometry><mesh filename="package://tool_manipulator_description/meshes/visual/tool1_drill.stl" scale="0.001 0.001 0.001"/></geometry><material name="motor_grey"/></visual>
