Commit message: Refactor tool manipulator configuration and update joint definitions
- Updated joint names in docking and simulation configurations to include wrist_pitch_joint and wrist_roll_joint.
- Adjusted joint goals and limits for the new joint configuration.
- Disabled gripper tools in tools.yaml and removed associated group states in SRDF.
- Modified launch files to use mock hardware for simulation.
- Added new collision meshes for various components of the tool manipulator.
- Introduced a mock hardware interface in the URDF for simulation purposes.

File: src/arm/tool_manipulator_description/urdf/tool_manipulator.urdf.xacro (robot description, xacro)
@@ -6,4 +6,5 @@
   <!-- ========================================================= -->
   <xacro:arg name="use_mesh" default="true"/>
+  <xacro:arg name="tool_id" default="0"/>
   <xacro:property
       name="mesh_path"
@@ -338,3 +339,18 @@
         rpy="0 0 0"/>
   </joint>
+  <!-- RealSense D435 bracket: TCP is the mechanical parent frame. -->
+  </link>
+    <link name="cam_link">
+    <xacro:mesh_visual
+        mesh="cam_d435"
+        material="motor_grey"/>
+  </link>
+  <joint name="cam_link_mount"
+         type="fixed">
+    <parent link="tcp_link"/>
+    <child link="cam_link"/>
+    <origin
+        xyz="0 0.0607680 0.074000"
+        rpy="${pi/2} 0 ${-pi/2}"/>
+  </joint>
 </robot>

File: src/arm/tool_manipulator_description/urdf/tool_manipulator_6dof_cad.urdf.xacro (robot description, xacro)
@@ -6,4 +6,5 @@
   <!-- ========================================================= -->
   <xacro:arg name="use_mesh" default="true"/>
+  <xacro:arg name="tool_id" default="0"/>
   <xacro:property
       name="mesh_path"
@@ -338,3 +339,17 @@
         rpy="0 0 0"/>
   </joint>
+  <!-- RealSense D435 bracket: TCP is the mechanical parent frame. -->
+  <joint name="tcp_to_cam_joint" type="fixed">
+    <parent link="tcp_link"/>
+    <child link="cam_link"/>
+    <origin xyz="0 0 0" rpy="0 0 0"/>
+  </joint>
+  <link name="cam_link">
+    <xacro:mesh_visual mesh="cam_d435" material="motor_grey"/>
+    <!-- Conservative D435/bracket envelope until a collision STL is supplied. -->
+    <collision>
+      <origin xyz="0 0 0" rpy="0 0 0"/>
+      <geometry><box size="0.025 0.090 0.025"/></geometry>
+    </collision>
+  </link>
 </robot>

File: src/arm/tool_manipulator_design_moveit_config/config/tool_manipulator.urdf.xacro (robot description, xacro)
@@ -1,4 +1,17 @@
 <?xml version="1.0"?>
 <robot xmlns:xacro="http://www.ros.org/wiki/xacro" name="tool_manipulator">
+  <xacro:arg name="use_mock_hardware" default="true"/>
+  <xacro:arg name="use_mesh" default="true"/>
   <xacro:include filename="$(find tool_manipulator_description)/urdf/tool_manipulator.urdf.xacro"/>
+  <!-- The CAD description has no hardware tag.  This self-contained mock
+       interface exists only for simulation and MoveIt integration. -->
+  <ros2_control name="ToolManipulatorMockSystem" type="system">
+    <hardware><plugin>mock_components/GenericSystem</plugin></hardware>
+    <joint name="base_joint"><command_interface name="position"/><state_interface name="position"><param name="initial_value">0</param></state_interface><state_interface name="velocity"/></joint>
+    <joint name="shoulder_joint"><command_interface name="position"/><state_interface name="position"><param name="initial_value">0</param></state_interface><state_interface name="velocity"/></joint>
+    <joint name="elbow_joint"><command_interface name="position"/><state_interface name="position"><param name="initial_value">0</param></state_interface><state_interface name="velocity"/></joint>
+    <joint name="wrist_pitch_joint"><command_interface name="position"/><state_interface name="position"><param name="initial_value">0</param></state_interface><state_interface name="velocity"/></joint>
+    <joint name="wrist_roll_joint"><command_interface name="position"/><state_interface name="position"><param name="initial_value">0</param></state_interface><state_interface name="velocity"/></joint>
+    <joint name="wrist_yaw_joint"><command_interface name="position"/><state_interface name="position"><param name="initial_value">0</param></state_interface><state_interface name="velocity"/></joint>
+  </ros2_control>
 </robot>

Commit message: fix: 수정된 카메라 링크 마운트의 부모 링크 및 회전 값

File: src/arm/tool_manipulator_description/urdf/tool_manipulator.urdf.xacro (robot description, xacro)
@@ -348,9 +348,9 @@
   <joint name="cam_link_mount"
          type="fixed">
-    <parent link="tcp_link"/>
+    <parent link="wrist_link_yaw"/>
     <child link="cam_link"/>
     <origin
         xyz="0 0.0607680 0.074000"
-        rpy="${pi/2} 0 ${-pi/2}"/>
+        rpy="${pi/2} ${pi} 0"/>
   </joint>
 </robot>

Commit message: feat: arm pose 캡처 스크립트 추가 및 CMake 및 패키지 의존성 업데이트

File: src/arm/tool_manipulator_description/urdf/tool_manipulator.urdf.xacro (robot description, xacro)
@@ -340,6 +340,5 @@
   </joint>
   <!-- RealSense D435 bracket: TCP is the mechanical parent frame. -->
-  </link>
-    <link name="cam_link">
+  <link name="cam_link">
     <xacro:mesh_visual
         mesh="cam_d435"

Commit message: Enhance tool manipulator URDF with new tools and configurations
- Added support for multiple tools (tool_1, tool_2, tool_3) in the tool manipulator URDF.
- Updated tool_2 and tool_3 definitions to include visual and collision meshes, along with proper inertial properties.
- Removed the tool group from the MoveIt SRDF configuration as it is no longer necessary.
- Introduced conditional inclusion of tools based on the selected tool ID, allowing for dynamic tool selection.

File: src/arm/tool_manipulator_description/urdf/tool_manipulator.urdf.xacro (robot description, xacro)
@@ -7,4 +7,8 @@
   <xacro:arg name="use_mesh" default="true"/>
   <xacro:arg name="tool_id" default="0"/>
+  <xacro:include filename="tools/tool_1_gripper.xacro"/>
+  <xacro:property name="selected_tool_id" value="$(arg tool_id)"/>
+  <xacro:include filename="tools/tool_2.xacro"/>
+  <xacro:include filename="tools/tool_3.xacro"/>
   <xacro:property
       name="mesh_path"
@@ -17,4 +21,7 @@
     <color rgba="0.20 0.20 0.22 1.0"/>
   </material>
+  <material name="petg_grey"><color rgba="0.40 0.40 0.42 1.0"/></material>
+  <material name="motor_dark"><color rgba="0.12 0.12 0.14 1.0"/></material>
+  <material name="tcp_red"><color rgba="0.90 0.05 0.05 1.0"/></material>
   <!-- MOTOR -->
   <material name="motor_grey">
@@ -353,3 +360,13 @@
         rpy="${-pi/2} ${-pi/2} 0"/>
   </joint>
+  <!-- The common arm ends at tcp_link; the selected tool is downstream. -->
+  <xacro:if value="${selected_tool_id == 1}">
+    <xacro:tool_1_gripper prefix="" parent="tcp_link" use_mesh="$(arg use_mesh)"/>
+  </xacro:if>
+  <xacro:if value="${selected_tool_id == 2}">
+    <xacro:tool_2 prefix="" parent="tcp_link" use_mesh="$(arg use_mesh)"/>
+  </xacro:if>
+  <xacro:if value="${selected_tool_id == 3}">
+    <xacro:tool_3 prefix="" parent="tcp_link" use_mesh="$(arg use_mesh)"/>
+  </xacro:if>
 </robot>

File: src/arm/tool_manipulator_description/urdf/tools/tool_2.xacro (robot description, xacro)
@@ -3,6 +3,10 @@
   <xacro:macro name="tool_2" params="prefix parent use_mesh:=false">
     <joint name="${prefix}tool_2_mount_joint" type="fixed"><parent link="${parent}"/><child link="${prefix}tool_2_link"/><origin xyz="0 0 0"/></joint>
-    <link name="${prefix}tool_2_link"><inertial><mass value="0.001"/><inertia ixx="1e-7" ixy="0" ixz="0" iyy="1e-7" iyz="0" izz="1e-7"/></inertial></link>
-    <joint name="${prefix}tool_2_tcp_joint" type="fixed"><parent link="${prefix}tool_2_link"/><child link="${prefix}tool_2_tcp"/><origin xyz="0 0 0"/></joint>
+    <link name="${prefix}tool_2_link">
+      <visual><geometry><mesh filename="package://tool_manipulator_description/meshes/visual/long_drillbit.stl" scale="0.001 0.001 0.001"/></geometry></visual>
+      <collision><geometry><mesh filename="package://tool_manipulator_description/meshes/collision/long_drillbit.stl" scale="0.001 0.001 0.001"/></geometry></collision>
+      <inertial><origin xyz="0 0.030 0"/><mass value="0.050"/><inertia ixx="0.00002" ixy="0" ixz="0" iyy="0.000004" iyz="0" izz="0.00002"/></inertial>
+    </link>
+    <joint name="${prefix}tool_2_tcp_joint" type="fixed"><parent link="${prefix}tool_2_link"/><child link="${prefix}tool_2_tcp"/><origin xyz="0 0.060 0"/></joint>
     <link name="${prefix}tool_2_tcp"/>
   </xacro:macro>

File: src/arm/tool_manipulator_description/urdf/tools/tool_3.xacro (robot description, xacro)
@@ -3,6 +3,10 @@
   <xacro:macro name="tool_3" params="prefix parent use_mesh:=false">
     <joint name="${prefix}tool_3_mount_joint" type="fixed"><parent link="${parent}"/><child link="${prefix}tool_3_link"/><origin xyz="0 0 0"/></joint>
-    <link name="${prefix}tool_3_link"><inertial><mass value="0.001"/><inertia ixx="1e-7" ixy="0" ixz="0" iyy="1e-7" iyz="0" izz="1e-7"/></inertial></link>
-    <joint name="${prefix}tool_3_tcp_joint" type="fixed"><parent link="${prefix}tool_3_link"/><child link="${prefix}tool_3_tcp"/><origin xyz="0 0 0"/></joint>
+    <link name="${prefix}tool_3_link">
+      <visual><geometry><mesh filename="package://tool_manipulator_description/meshes/visual/long_phillipsbit.stl" scale="0.001 0.001 0.001"/></geometry></visual>
+      <collision><geometry><mesh filename="package://tool_manipulator_description/meshes/collision/long_phillipsbit.stl" scale="0.001 0.001 0.001"/></geometry></collision>
+      <inertial><origin xyz="0 0.0283 0"/><mass value="0.050"/><inertia ixx="0.00002" ixy="0" ixz="0" iyy="0.000004" iyz="0" izz="0.00002"/></inertial>
+    </link>
+    <joint name="${prefix}tool_3_tcp_joint" type="fixed"><parent link="${prefix}tool_3_link"/><child link="${prefix}tool_3_tcp"/><origin xyz="0 0.0508 0"/></joint>
     <link name="${prefix}tool_3_tcp"/>
   </xacro:macro>

Commit message: feat: add tool attachment manager and enhance docking functionality
- Added tool_attachment_manager.py to manage physical tool changes in the MoveIt planning scene.
- Updated apriltag_tool_docking_node.py to handle new docking states and integrate with the tool attachment manager.
- Modified docking.yaml and tools.yaml to include new parameters for tool attachment and docking behavior.
- Enhanced CMakeLists.txt to install the new tool_attachment_manager script.
- Removed outdated TODO.md file.
- Updated URDF and XACRO files for tools to reflect new configurations and limits.
- Added new launch file tool_demo.launch.py for offline MoveIt inspection with static tool models.
- Updated collision and visual mesh files for long drill bit and long Phillips bit.

File: src/arm/tool_manipulator_description/urdf/tool_manipulator.urdf.xacro (robot description, xacro)
@@ -262,8 +262,8 @@
     <axis xyz="0 0 1"/>
     <limit
-        lower="${-pi}"
-        upper="${pi}"
-        effort="1.0"
-        velocity="1.0"/>
+        lower="-0.894310799337"
+        upper="0.567572891518"
+        effort="1.0"
+        velocity="5.035176563244"/>
   </joint>
   <!-- ========================================================= -->

File: src/arm/tool_manipulator_description/urdf/tools/tool_1_gripper.xacro (robot description, xacro)
@@ -5,4 +5,8 @@
   <xacro:macro name="tool_1_gripper" params="prefix parent use_mesh:=false">
     <xacro:property name="tool_1_tcp_offset" value="0.090"/>
+    <!-- MX-106 raw reference: raw 0 = 0 rad; raw increment = CCW/closing; 4096 tick/rev. -->
+    <xacro:property name="tool_1_gripper_limit_lower" value="-1.279339977097"/> <!-- raw 459; raw 1293 = 0 -->
+    <xacro:property name="tool_1_gripper_open" value="0.0"/> <!-- raw 1293: open reference -->
+    <xacro:property name="tool_1_gripper_limit_upper" value="3.911651009108"/> <!-- raw 3843 -->
     <xacro:property name="tool_1_rack_offset" value="0.018"/>
     <xacro:property name="tool_1_pitch_radius" value="0.017"/>
@@ -14,27 +18,19 @@
       <inertial><mass value="0.001"/><inertia ixx="1e-7" ixy="0" ixz="0" iyy="1e-7" iyz="0" izz="1e-7"/></inertial>
     </link>
+    <!-- Common tool geometry frame: from tcp_link, rotate Y +90 deg then Z +90 deg. -->
+    <joint name="${prefix}tool_1_geometry_joint" type="fixed">
+      <parent link="${prefix}tool_1_link"/><child link="${prefix}tool_1_geometry_link"/>
+      <origin xyz="0 0 0" rpy="0 ${pi/2} ${pi/2}"/>
+    </joint>
+    <link name="${prefix}tool_1_geometry_link"/>
     <!-- ========== gripper_actuator -> pinion_gear (revolute, "피니언 구동") ==========-->
     <joint name="${prefix}gripper_joint" type="revolute">
-      <parent link="${prefix}ee_actuator"/>
+      <parent link="${prefix}tool_1_geometry_link"/>
       <child  link="${prefix}pinion_gear"/>
-      <origin xyz=" 0 0 0" rpy="0 0 0"/>
+      <origin xyz="0 0 0" rpy="0 ${pi/2} 0"/>
       <axis xyz="0 0 1"/>
-      <limit lower="${gripper_limit_lower}" upper="${gripper_limit_upper}" effort="8.4" velocity="3.665"/>
+      <limit lower="${tool_1_gripper_limit_lower}" upper="${tool_1_gripper_limit_upper}" effort="8.4" velocity="3.665"/>
       <dynamics damping="0.05" friction="0.01"/>
     </joint>
-    <!-- gripper_actuator: MX-106T stator, wrist_link의 형제(fixed) 링크. -->
-    <joint name="${prefix}gripper_actuator_joint" type="fixed">
-      <parent link="${prefix}wrist_link_yaw"/>
-      <child link="${prefix}ee_actuator"/>
-      <origin xyz="-${L3} 0 ${-off_wrist}" rpy="0 -${pi/2} 0"/>
-    </joint>
-    <link name="${prefix}gripper_actuator">
-      <xacro:if value="${use_mesh}">
-        <visual><origin xyz="0 0 0" rpy="0 0 ${pi/2}"/><geometry><mesh filename="package:/tool_manipulator_description/meshes/visual/ee_actuator.stl" scale="0.001 0.001 0.001"/></geometry><material name="motor_dark"/></visual>
-        <collision><origin xyz="0 0 0" rpy="0 0 ${pi/2}"/><geometry><mesh filename="package://tool_manipulator_description/meshes/collision/ee_actuator.stl" scale="0.001 0.001 0.001"/></geometry></collision>
-      </xacro:if>
-      <xacro:unless value="${use_mesh}"><visual><geometry><cylinder radius="0.030" length="0.050"/></geometry><material name="motor_dark"/></visual><collision><geometry><cylinder radius="0.030" length="0.050"/></geometry></collision></xacro:unless>
-      <inertial><mass value="0.001"/><inertia ixx="1e-7" ixy="0" ixz="0" iyy="1e-7" iyz="0" izz="1e-7"/></inertial>
-    </link>
     <!-- pinion_gear: m=1, z=34, 피치반경 17mm (module 1 x teeth 34 / 2, 2026-08-30 mesh 개정) -->
     <link name="${prefix}pinion_gear">
@@ -69,5 +65,5 @@
     <!-- ========== wrist_link -> rack_left (prismatic, mimic) ==========-->
     <joint name="${prefix}rack_left_joint" type="prismatic">
-      <parent link="${prefix}wrist_link"/>
+      <parent link="${prefix}tool_1_geometry_link"/>
       <child  link="${prefix}rack_left"/>
       <xacro:property name="pinion_pitch_radius" value="0.017"/>
@@ -75,5 +71,5 @@
            기존에는 wrist_link의 z=0을 중심으로 ±0.062를 줘서 pinion_gear
            원점(z=${-off_wrist})만큼 어긋나 있었음 - 2026-08-24 수정. -->
-      <origin xyz="${-L3} 0.018 ${-off_wrist + 0.062}" rpy="${pi} 0 ${pi}"/>
+      <origin xyz="-0.016 0.018 0.062" rpy="${pi} 0 ${pi}"/>
       <axis xyz="0 0 1"/>
       <limit lower="0" upper="0.030" effort="8.4" velocity="0.1"/>
@@ -119,9 +115,9 @@
     <!-- ========== wrist_link -> rack_right (prismatic, mimic, 반대방향) ==========-->
     <joint name="${prefix}rack_right_joint" type="prismatic">
-      <parent link="${prefix}wrist_link"/>
+      <parent link="${prefix}tool_1_geometry_link"/>
       <child  link="${prefix}rack_right"/>
       <!-- z: pinion_gear 원점(wrist_link 기준 z=${-off_wrist})에서 -0.062 오프셋.
            rack_left_joint와 동일한 수정 - 2026-08-24. -->
-      <origin xyz="${-L3} -0.018 ${-off_wrist - 0.062}" rpy="0 0 0"/>
+      <origin xyz="-0.016 -0.018 -0.062" rpy="0 0 0"/>
       <axis xyz="0 0 1"/>
       <limit lower="0" upper="0.030" effort="8.4" velocity="0.1"/>
@@ -159,3 +155,4 @@
       </inertial>
     </link>
+  </xacro:macro>
 </robot>

File: src/arm/tool_manipulator_description/urdf/tools/tool_2.xacro (robot description, xacro)
@@ -2,7 +2,7 @@
 <robot xmlns:xacro="http://www.ros.org/wiki/xacro">
   <xacro:macro name="tool_2" params="prefix parent use_mesh:=false">
-    <joint name="${prefix}tool_2_mount_joint" type="fixed"><parent link="${parent}"/><child link="${prefix}tool_2_link"/><origin xyz="0 0 0"/></joint>
+    <joint name="${prefix}tool_2_mount_joint" type="fixed"><parent link="${parent}"/><child link="${prefix}tool_2_link"/><origin xyz="0 0 0.012" rpy="${pi/2} 0 0"/></joint>
     <link name="${prefix}tool_2_link">
-      <visual><geometry><mesh filename="package://tool_manipulator_description/meshes/visual/long_drillbit.stl" scale="0.001 0.001 0.001"/></geometry></visual>
+      <visual><geometry><mesh filename="package://tool_manipulator_description/meshes/visual/long_drillbit.stl" scale="0.001 0.001 0.001"/></geometry><material name="motor_grey"/></visual>
       <collision><geometry><mesh filename="package://tool_manipulator_description/meshes/collision/long_drillbit.stl" scale="0.001 0.001 0.001"/></geometry></collision>
       <inertial><origin xyz="0 0.030 0"/><mass value="0.050"/><inertia ixx="0.00002" ixy="0" ixz="0" iyy="0.000004" iyz="0" izz="0.00002"/></inertial>

File: src/arm/tool_manipulator_description/urdf/tools/tool_3.xacro (robot description, xacro)
@@ -2,7 +2,7 @@
 <robot xmlns:xacro="http://www.ros.org/wiki/xacro">
   <xacro:macro name="tool_3" params="prefix parent use_mesh:=false">
-    <joint name="${prefix}tool_3_mount_joint" type="fixed"><parent link="${parent}"/><child link="${prefix}tool_3_link"/><origin xyz="0 0 0"/></joint>
+    <joint name="${prefix}tool_3_mount_joint" type="fixed"><parent link="${parent}"/><child link="${prefix}tool_3_link"/><origin xyz="0 0 0.015" rpy="${pi/2} 0 0"/></joint>
     <link name="${prefix}tool_3_link">
-      <visual><geometry><mesh filename="package://tool_manipulator_description/meshes/visual/long_phillipsbit.stl" scale="0.001 0.001 0.001"/></geometry></visual>
+      <visual><geometry><mesh filename="package://tool_manipulator_description/meshes/visual/long_phillipsbit.stl" scale="0.001 0.001 0.001"/></geometry><material name="motor_grey"/></visual>
       <collision><geometry><mesh filename="package://tool_manipulator_description/meshes/collision/long_phillipsbit.stl" scale="0.001 0.001 0.001"/></geometry></collision>
       <inertial><origin xyz="0 0.0283 0"/><mass value="0.050"/><inertia ixx="0.00002" ixy="0" ixz="0" iyy="0.000004" iyz="0" izz="0.00002"/></inertial>
