Commit message: feat: Add visual servo node for XY-only control and update URDF/XACRO files
- Introduced a new `visual_servo_node.py` script for handling visual servoing based on tag pose filtering.
- Updated `display.launch.py` to change the joint name from `gripper_joint` to `ee_joint`.
- Modified `tool_manipulator.urdf.xacro` to include chassis dimensions and new materials, and added collision geometry for the tool manipulator.
- Updated `tool_1_gripper.xacro` to replace `gripper_joint` with `ee_joint` for better integration with the new end-effector structure.
- Enhanced `ros2_controllers.yaml` to include an `ee_controller` for the end-effector joint.
- Updated `tool_manipulator.ros2_control.xacro` to define the end-effector joint and integrate it with the existing control structure.
- Adjusted `tool_manipulator.urdf.xacro` to streamline the inclusion of control configurations and initial positions.
- Updated package dependencies in `package.xml` to include necessary controllers and hardware interfaces.
- Corrected the directory path in `howtorun.md` for running tests.

File: src/arm/tool_manipulator_moveit_config/config/tool_manipulator.ros2_control.xacro (robot description, xacro)
@@ -1,54 +1,109 @@
 <?xml version="1.0"?>
 <robot xmlns:xacro="http://www.ros.org/wiki/xacro">
-    <xacro:macro name="tool_manipulator_ros2_control" params="name initial_positions_file">
-        <xacro:property name="initial_positions" value="${load_yaml(initial_positions_file)['initial_positions']}"/>
-        <ros2_control name="${name}" type="system">
-            <hardware>
-                <!-- By default, set up controllers for simulation. This won't work on real hardware -->
-                <plugin>mock_components/GenericSystem</plugin>
-            </hardware>
-            <joint name="base_joint">
-                <command_interface name="position"/>
-                <state_interface name="position">
-                  <param name="initial_value">${initial_positions['base_joint']}</param>
-                </state_interface>
-                <state_interface name="velocity"/>
-            </joint>
-            <joint name="shoulder_joint">
-                <command_interface name="position"/>
-                <state_interface name="position">
-                  <param name="initial_value">${initial_positions['shoulder_joint']}</param>
-                </state_interface>
-                <state_interface name="velocity"/>
-            </joint>
-            <joint name="elbow_joint">
-                <command_interface name="position"/>
-                <state_interface name="position">
-                  <param name="initial_value">${initial_positions['elbow_joint']}</param>
-                </state_interface>
-                <state_interface name="velocity"/>
-            </joint>
-            <joint name="wrist_pitch_joint">
-                <command_interface name="position"/>
-                <state_interface name="position">
-                  <param name="initial_value">${initial_positions['wrist_pitch_joint']}</param>
-                </state_interface>
-                <state_interface name="velocity"/>
-            </joint>
-            <joint name="wrist_roll_joint">
-                <command_interface name="position"/>
-                <state_interface name="position">
-                  <param name="initial_value">${initial_positions['wrist_roll_joint']}</param>
-                </state_interface>
-                <state_interface name="velocity"/>
-            </joint>
-            <joint name="wrist_yaw_joint">
-                <command_interface name="position"/>
-                <state_interface name="position">
-                  <param name="initial_value">${initial_positions['wrist_yaw_joint']}</param>
-                </state_interface>
-                <state_interface name="velocity"/>
-            </joint>
-        </ros2_control>
-    </xacro:macro>
+  <!-- FakeSystem is retained for offline planning only. The real branch consumes
+       tool_manipulator_bringup/config/hardware.yaml after preflight succeeds. -->
+  <xacro:macro name="fake_joint" params="name initial">
+    <joint name="${name}">
+      <command_interface name="position"/>
+      <state_interface name="position"><param name="initial_value">${initial}</param></state_interface>
+      <state_interface name="velocity"/>
+    </joint>
+  </xacro:macro>
+  <xacro:macro name="rmd_actuator" params="name spec can_ifname">
+    <ros2_control name="rmd_${name}" type="actuator">
+      <hardware>
+        <plugin>rmd_hardware_interface/MyActuatorRmdHardwareInterface</plugin>
+        <param name="ifname">${can_ifname}</param>
+        <param name="actuator_id">${spec['id']}</param>
+        <param name="sign">${spec['sign']}</param>
+        <param name="q_offset">${spec['q_offset_rad']}</param>
+        <param name="max_velocity">${spec['velocity_limit_rad_s']}</param>
+        <param name="software_current_limit">${spec['current_limit_a']}</param>
+        <param name="current_release_threshold">${spec['current_release_threshold_a']}</param>
+        <param name="current_retreat_velocity">${spec['current_retreat_velocity_rad_s']}</param>
+        <param name="current_max_retreat_distance">${spec['current_max_retreat_distance_rad']}</param>
+        <param name="current_limit_duration_ms">${spec['current_limit_duration_ms']}</param>
+        <param name="velocity_alpha">0.1</param>
+        <param name="effort_alpha">0.1</param>
+        <param name="can_receive_timeout_ms">100</param>
+        <param name="initial_feedback_timeout_ms">3000</param>
+        <param name="feedback_timeout_ms">500</param>
+        <param name="position_limit_rejection_margin">0.01745329252</param>
+      </hardware>
+      <joint name="${name}">
+        <command_interface name="position" min="${spec['soft_limit_rad'][0]}" max="${spec['soft_limit_rad'][1]}"/>
+        <state_interface name="position"/><state_interface name="velocity"/><state_interface name="effort"/>
+      </joint>
+    </ros2_control>
+  </xacro:macro>
+  <xacro:macro name="dxl_joint" params="name spec wrap">
+    <joint name="${name}">
+      <command_interface name="position" min="${spec['soft_limit_rad'][0]}" max="${spec['soft_limit_rad'][1]}"/>
+      <state_interface name="position"/><state_interface name="velocity"/><state_interface name="effort"/>
+      <!-- Model coordinate is raw_tick*2pi/4096-pi. -->
+      <param name="position_zero_offset">${spec['zero_raw'] * 2.0 * pi / 4096.0 - pi}</param>
+      <param name="position_direction">1.0</param>
+      <param name="position_wraparound">${wrap}</param>
+    </joint>
+  </xacro:macro>
+  <xacro:macro name="dxl_gpio" params="name spec">
+    <gpio name="${name}">
+      <param name="type">dxl</param><param name="ID">${spec['id']}</param>
+      <param name="transport_channel">${spec['transport_channel']}</param>
+      <command_interface name="Goal Position"/>
+      <state_interface name="Present Position"/><state_interface name="Present Velocity"/><state_interface name="Present Current"/>
+      <param name="Operating Mode">${spec['operating_mode']}</param>
+      <param name="Current Limit">${spec['current_limit_raw']}</param>
+      <param name="Velocity Limit">${spec['velocity_limit_raw']}</param>
+      <param name="Profile Acceleration">${spec['profile_acceleration_raw']}</param>
+      <param name="Profile Velocity">${spec['profile_velocity_raw']}</param>
+    </gpio>
+  </xacro:macro>
+  <xacro:macro name="tool_manipulator_ros2_control" params="name initial_positions_file use_mock_hardware:=true hardware_config_file:=''">
+    <xacro:property name="initial_positions" value="${load_yaml(initial_positions_file)['initial_positions']}"/>
+    <xacro:if value="${use_mock_hardware}">
+      <ros2_control name="${name}" type="system"><hardware><plugin>mock_components/GenericSystem</plugin></hardware>
+        <xacro:fake_joint name="base_joint" initial="${initial_positions['base_joint']}"/>
+        <xacro:fake_joint name="shoulder_joint" initial="${initial_positions['shoulder_joint']}"/>
+        <xacro:fake_joint name="elbow_joint" initial="${initial_positions['elbow_joint']}"/>
+        <xacro:fake_joint name="wrist_pitch_joint" initial="${initial_positions['wrist_pitch_joint']}"/>
+        <xacro:fake_joint name="wrist_roll_joint" initial="${initial_positions['wrist_roll_joint']}"/>
+        <xacro:fake_joint name="wrist_yaw_joint" initial="${initial_positions['wrist_yaw_joint']}"/>
+        <xacro:fake_joint name="ee_joint" initial="0.0"/>
+      </ros2_control>
+    </xacro:if>
+    <xacro:unless value="${use_mock_hardware}">
+      <xacro:property name="hw" value="${load_yaml(hardware_config_file)}"/>
+      <xacro:property name="j" value="${hw['joints']}"/>
+      <!-- One U2D2 serial device owns the confirmed TTL + RS-485 chains. -->
+      <ros2_control name="dynamixel_u2d2" type="system">
+        <hardware>
+          <plugin>dynamixel_hardware_interface/DynamixelHardware</plugin>
+          <param name="number_of_joints">4</param><param name="number_of_transmissions">4</param>
+          <param name="port_name">${hw['buses']['dynamixel_u2d2']['device']}</param>
+          <param name="baud_rate">${hw['buses']['dynamixel_u2d2']['baud_rate']}</param>
+          <param name="u2d2_mixed_ttl_rs485">${hw['buses']['dynamixel_u2d2']['mixed_ttl_rs485']}</param>
+          <param name="feedback_mode">${hw['buses']['dynamixel_u2d2']['feedback_mode']}</param>
+          <param name="command_mode">${hw['buses']['dynamixel_u2d2']['command_mode']}</param>
+          <param name="dynamixel_model_folder">/param/dxl_model</param>
+          <param name="disable_torque_at_init">true</param>
+          <param name="error_timeout_ms">500</param>
+          <param name="position_limit_rejection_margin">0.01745329252</param>
+          <param name="transmission_to_joint_matrix">1,0,0,0,0,1,0,0,0,0,1,0,0,0,0,1</param>
+          <param name="joint_to_transmission_matrix">1,0,0,0,0,1,0,0,0,0,1,0,0,0,0,1</param>
+        </hardware>
+        <xacro:dxl_joint name="base_joint" spec="${j['base_joint']}" wrap="true"/>
+        <xacro:dxl_joint name="wrist_roll_joint" spec="${j['wrist_roll_joint']}" wrap="false"/>
+        <xacro:dxl_joint name="wrist_yaw_joint" spec="${j['wrist_yaw_joint']}" wrap="true"/>
+        <xacro:dxl_joint name="ee_joint" spec="${j['ee_joint']}" wrap="false"/>
+        <xacro:dxl_gpio name="base_motor" spec="${j['base_joint']}"/>
+        <xacro:dxl_gpio name="wrist_roll_motor" spec="${j['wrist_roll_joint']}"/>
+        <xacro:dxl_gpio name="wrist_yaw_motor" spec="${j['wrist_yaw_joint']}"/>
+        <xacro:dxl_gpio name="ee_motor" spec="${j['ee_joint']}"/>
+      </ros2_control>
+      <xacro:rmd_actuator name="shoulder_joint" spec="${j['shoulder_joint']}" can_ifname="${hw['buses']['rmd_can']['interface']}"/>
+      <xacro:rmd_actuator name="elbow_joint" spec="${j['elbow_joint']}" can_ifname="${hw['buses']['rmd_can']['interface']}"/>
+      <xacro:rmd_actuator name="wrist_pitch_joint" spec="${j['wrist_pitch_joint']}" can_ifname="${hw['buses']['rmd_can']['interface']}"/>
+    </xacro:unless>
+  </xacro:macro>
 </robot>

File: src/arm/tool_manipulator_moveit_config/config/tool_manipulator.urdf.xacro (robot description, xacro)
@@ -1,9 +1,9 @@
 <?xml version="1.0"?>
 <robot xmlns:xacro="http://www.ros.org/wiki/xacro" name="tool_manipulator">
-    <xacro:arg name="initial_positions_file" default="initial_positions.yaml" />
-    <!-- Import tool_manipulator urdf file -->
-    <xacro:include filename="$(find tool_manipulator_description)/urdf/tool_manipulator.urdf.xacro" />
-    <!-- Import control_xacro -->
-    <xacro:include filename="tool_manipulator.ros2_control.xacro" />
-    <xacro:tool_manipulator_ros2_control name="FakeSystem" initial_positions_file="$(arg initial_positions_file)"/>
+  <xacro:arg name="initial_positions_file" default="initial_positions.yaml"/>
+  <xacro:arg name="use_mock_hardware" default="true"/>
+  <xacro:arg name="hardware_config_file" default=""/>
+  <xacro:include filename="$(find tool_manipulator_description)/urdf/tool_manipulator.urdf.xacro"/>
+  <xacro:include filename="tool_manipulator.ros2_control.xacro"/>
+  <xacro:tool_manipulator_ros2_control name="tool_manipulator_system" initial_positions_file="$(arg initial_positions_file)" use_mock_hardware="$(arg use_mock_hardware)" hardware_config_file="$(arg hardware_config_file)"/>
 </robot>

Commit message: feat: Update tool case dimensions and entry specifications in URDF

File: src/arm/tool_manipulator_description/urdf/tool_manipulator.urdf.xacro (robot description, xacro)
@@ -112,14 +112,14 @@
     <origin xyz="$(arg arm_world_x) $(arg arm_world_y) $(arg arm_world_z)" rpy="0 0 0"/>
   </joint>
-  <!-- Tool-case outer: 36.8 x 46.8 x 50 mm; insertion void: 16 x 16 x 50 mm. -->
+  <!-- Case 2/3 outer: 36.8(X) x 46.8(Y) x 50(Z) mm.
+       EE entry is local +X; cavity is 16(X depth) x 16(Y) x 50(Z) mm. -->
   <xacro:macro name="tool_case_walls">
-    <visual><origin xyz="-0.0132 0 0"/><geometry><box size="0.0104 0.0468 0.050"/></geometry><material name="tool_case_blue"/></visual>
-    <collision><origin xyz="-0.0132 0 0"/><geometry><box size="0.0104 0.0468 0.050"/></geometry></collision>
-    <visual><origin xyz="0.0132 0 0"/><geometry><box size="0.0104 0.0468 0.050"/></geometry><material name="tool_case_blue"/></visual>
-    <collision><origin xyz="0.0132 0 0"/><geometry><box size="0.0104 0.0468 0.050"/></geometry></collision>
-    <visual><origin xyz="0 -0.0157 0"/><geometry><box size="0.0160 0.0154 0.050"/></geometry><material name="tool_case_blue"/></visual>
-    <collision><origin xyz="0 -0.0157 0"/><geometry><box size="0.0160 0.0154 0.050"/></geometry></collision>
-    <visual><origin xyz="0 0.0157 0"/><geometry><box size="0.0160 0.0154 0.050"/></geometry><material name="tool_case_blue"/></visual>
-    <collision><origin xyz="0 0.0157 0"/><geometry><box size="0.0160 0.0154 0.050"/></geometry></collision>
+    <!-- back wall and two Y rails: open local +X face toward the EE -->
+    <visual><origin xyz="-0.008 0 0"/><geometry><box size="0.0208 0.0468 0.050"/></geometry><material name="tool_case_blue"/></visual>
+    <collision><origin xyz="-0.008 0 0"/><geometry><box size="0.0208 0.0468 0.050"/></geometry></collision>
+    <visual><origin xyz="0.0104 -0.0157 0"/><geometry><box size="0.016 0.0154 0.050"/></geometry><material name="tool_case_blue"/></visual>
+    <collision><origin xyz="0.0104 -0.0157 0"/><geometry><box size="0.016 0.0154 0.050"/></geometry></collision>
+    <visual><origin xyz="0.0104 0.0157 0"/><geometry><box size="0.016 0.0154 0.050"/></geometry><material name="tool_case_blue"/></visual>
+    <collision><origin xyz="0.0104 0.0157 0"/><geometry><box size="0.016 0.0154 0.050"/></geometry></collision>
   </xacro:macro>
   <!-- Case 2 (+Y) and case 3 (-Y) centres are arm_world offsets. Their Z
@@ -182,5 +182,5 @@
     <parent link="arm_world"/><child link="tool_case_1"/>
     <!-- arm_world has world orientation, so pitch +55 deg is world-Y tilt. -->
-    <origin xyz="-0.368 0 0.187" rpy="0 0.959931088597 0"/>
+    <origin xyz="-0.468 0 0.187" rpy="0 0.959931088597 0"/>
   </joint>
   <!-- Case-1 local YZ outer faces, at X = +/-18.4 mm. The positive face is the EE entry. -->

Commit message: feat: Update joint origin for tool_case_1 in URDF

File: src/arm/tool_manipulator_description/urdf/tool_manipulator.urdf.xacro (robot description, xacro)
@@ -182,5 +182,5 @@
     <parent link="arm_world"/><child link="tool_case_1"/>
     <!-- arm_world has world orientation, so pitch +55 deg is world-Y tilt. -->
-    <origin xyz="-0.468 0 0.187" rpy="0 0.959931088597 0"/>
+    <origin xyz="-0.427272082 0 0.190020943" rpy="0 0.959931088597 0"/>
   </joint>
   <!-- Case-1 local YZ outer faces, at X = +/-18.4 mm. The positive face is the EE entry. -->

Commit message: feat: 각 포즈 추가

File: src/arm/tool_manipulator_description/urdf/tool_manipulator.urdf.xacro (robot description, xacro)
@@ -228,6 +228,6 @@
     <!-- 임시 limit -->
     <limit
-        lower="${-pi}"
-        upper="${pi}"
+        lower="-3.503612119531"
+        upper="3.614058736259"
         effort="1.0"
         velocity="1.0"/>
@@ -271,6 +271,6 @@
     <axis xyz="0 0 -1"/>
     <limit
-        lower="${-pi}"
-        upper="${pi}"
+        lower="-1.459444233251"
+        upper="1.534842544204"
         effort="1.0"
         velocity="1.0"/>
@@ -314,6 +314,6 @@
     <axis xyz="0 0 -1"/>
     <limit
-        lower="${-pi}"
-        upper="${pi}"
+        lower="-1.475675812748"
+        upper="1.573239770294"
         effort="1.0"
         velocity="1.0"/>
@@ -357,6 +357,6 @@
     <axis xyz="0 0 -1"/>
     <limit
-        lower="${-pi}"
-        upper="${pi}"
+        lower="-1.643751229155"
+        upper="1.666265854332"
         effort="1.0"
         velocity="1.0"/>
@@ -400,6 +400,6 @@
     <axis xyz="0 0 1"/>
     <limit
-        lower="-0.894310799337"
-        upper="0.567572891518"
+        lower="-0.866699145155"
+        upper="0.688757373761"
         effort="1.0"
         velocity="5.035176563244"/>
@@ -443,6 +443,6 @@
     <axis xyz="0 0 1"/>
     <limit
-        lower="${-pi}"
-        upper="${pi}"
+        lower="-3.113980999408"
+        upper="3.156932461469"
         effort="1.0"
         velocity="1.0"/>

File: src/arm/tool_manipulator_moveit_config/config/tool_manipulator.ros2_control.xacro (robot description, xacro)
@@ -43,5 +43,5 @@
       <!-- Model coordinate is raw_tick*2pi/4096-pi. -->
       <param name="position_zero_offset">${spec['zero_raw'] * 2.0 * pi / 4096.0 - pi}</param>
-      <param name="position_direction">1.0</param>
+      <param name="position_direction">${1.0 if spec['raw_increases_ccw'] else -1.0}</param>
       <param name="position_wraparound">${wrap}</param>
     </joint>
@@ -61,5 +61,5 @@
   </xacro:macro>
   <xacro:macro name="tool_manipulator_ros2_control" params="name initial_positions_file use_mock_hardware:=true hardware_config_file:=''">
-    <xacro:property name="initial_positions" value="${load_yaml(initial_positions_file)['initial_positions']}"/>
+    <xacro:property name="initial_positions" value="${xacro.load_yaml(initial_positions_file)['initial_positions']}"/>
     <xacro:if value="${use_mock_hardware}">
       <ros2_control name="${name}" type="system"><hardware><plugin>mock_components/GenericSystem</plugin></hardware>
@@ -74,5 +74,5 @@
     </xacro:if>
     <xacro:unless value="${use_mock_hardware}">
-      <xacro:property name="hw" value="${load_yaml(hardware_config_file)}"/>
+      <xacro:property name="hw" value="${xacro.load_yaml(hardware_config_file)}"/>
       <xacro:property name="j" value="${hw['joints']}"/>
       <!-- One U2D2 serial device owns the confirmed TTL + RS-485 chains. -->
@@ -93,7 +93,7 @@
           <param name="joint_to_transmission_matrix">1,0,0,0,0,1,0,0,0,0,1,0,0,0,0,1</param>
         </hardware>
-        <xacro:dxl_joint name="base_joint" spec="${j['base_joint']}" wrap="true"/>
+        <xacro:dxl_joint name="base_joint" spec="${j['base_joint']}" wrap="false"/>
         <xacro:dxl_joint name="wrist_roll_joint" spec="${j['wrist_roll_joint']}" wrap="false"/>
-        <xacro:dxl_joint name="wrist_yaw_joint" spec="${j['wrist_yaw_joint']}" wrap="true"/>
+        <xacro:dxl_joint name="wrist_yaw_joint" spec="${j['wrist_yaw_joint']}" wrap="false"/>
         <xacro:dxl_joint name="ee_joint" spec="${j['ee_joint']}" wrap="false"/>
         <xacro:dxl_gpio name="base_motor" spec="${j['base_joint']}"/>

Commit message: 실측값 추가

File: src/arm/tool_manipulator_description/urdf/tool_manipulator.urdf.xacro (robot description, xacro)
@@ -491,6 +491,6 @@
     <parent link="tcp_link"/><child link="ee_output_link"/>
     <origin xyz="0 0 0" rpy="0 0 0"/><axis xyz="0 0 1"/>
-    <!-- raw 1293 = 0 rad; raw 459..3843 are the measured safe endpoints. -->
-    <limit lower="-1.279339977097" upper="3.911651009108" effort="8.4" velocity="5.035177"/>
+    <!-- raw 1992 = 0 rad; raw 459..3843 are the measured safe endpoints. -->
+    <limit lower="-2.351592547829" upper="2.839398438376" effort="8.4" velocity="5.035177"/>
   </joint>
   <!-- RealSense D435 bracket: TCP is the mechanical parent frame. -->

File: src/arm/tool_manipulator_description/urdf/tools/tool_1_gripper.xacro (robot description, xacro)
@@ -5,8 +5,9 @@
   <xacro:macro name="tool_1_gripper" params="prefix parent use_mesh:=false">
     <xacro:property name="tool_1_tcp_offset" value="0.090"/>
-    <!-- MX-106 raw reference: raw 0 = 0 rad; raw increment = CCW/closing; 4096 tick/rev. -->
-    <xacro:property name="tool_1_gripper_limit_lower" value="-1.279339977097"/> <!-- raw 459; raw 1293 = 0 -->
-    <xacro:property name="tool_1_gripper_open" value="0.0"/> <!-- raw 1293: open reference -->
-    <xacro:property name="tool_1_gripper_limit_upper" value="3.911651009108"/> <!-- raw 3843 -->
+    <!-- MX-106 raw reference: raw 1992 = 0 rad; raw increment = CCW/closing; 4096 tick/rev. -->
+    <xacro:property name="tool_1_gripper_limit_lower" value="-2.351592547829"/> <!-- raw 459 -->
+    <xacro:property name="tool_1_gripper_open" value="-0.076699"/> <!-- measured raw 1941..1942 -->
+    <xacro:property name="tool_1_gripper_close" value="1.251728"/> <!-- measured raw 2808 -->
+    <xacro:property name="tool_1_gripper_limit_upper" value="2.839398438376"/> <!-- raw 3843 -->
     <xacro:property name="tool_1_rack_offset" value="0.018"/>
     <xacro:property name="tool_1_pitch_radius" value="0.017"/>
@@ -76,5 +77,6 @@
            부호까지 반대로 주면 world 기준으로는 오히려 같은 방향으로 움직여
            버린다(실기에서 "한 몸으로 움직인다"고 확인된 원인). -->
-      <mimic joint="ee_joint" multiplier="${pinion_pitch_radius}" offset="0"/>
+      <mimic joint="ee_joint" multiplier="${pinion_pitch_radius}"
+             offset="${-tool_1_gripper_open * pinion_pitch_radius}"/>
     </joint>
     <link name="${prefix}rack_left">
@@ -119,5 +121,6 @@
       <axis xyz="0 0 1"/>
       <limit lower="0" upper="0.030" effort="8.4" velocity="0.1"/>
-      <mimic joint="ee_joint" multiplier="${pinion_pitch_radius}" offset="0"/>
+      <mimic joint="ee_joint" multiplier="${pinion_pitch_radius}"
+             offset="${-tool_1_gripper_open * pinion_pitch_radius}"/>
     </joint>
     <link name="${prefix}rack_right">
