Commit message: controlnode수정

File: src/arm/tool_manipulator_description/urdf/tool_manipulator.urdf.xacro (robot description, xacro)
@@ -123,6 +123,6 @@
     <collision><origin xyz="0.0104 0.0157 0"/><geometry><box size="0.016 0.0154 0.050"/></geometry></collision>
   </xacro:macro>
-  <!-- Case 2 (+Y) and case 3 (-Y) centres are arm_world offsets. Their Z
-       centres are calibrated so the tilted local +Z outer-face midpoint is
+  <!-- Case 2 (+Y) centre is an arm_world offset. Its Z
+       centre is calibrated so the tilted local +Z outer-face midpoint is
        z=167.935 mm in arm_world. -->
   <link name="tool_case_y_plus"><xacro:tool_case_walls/></link>
@@ -145,19 +145,10 @@
     <origin xyz="-0.0184 0 0" rpy="0 -1.570796326795 0"/>
   </joint>
-  <link name="tool_case_y_minus"><xacro:tool_case_walls/></link>
-  <joint name="arm_world_to_tool_case_y_minus" type="fixed">
-    <parent link="arm_world"/><child link="tool_case_y_minus"/>
-    <!-- arm_world has world orientation, so pitch +55 deg is world-Y tilt. -->
-    <origin xyz="-0.268 -0.10245 0.153595589" rpy="0 0.959931088597 0"/>
-  </joint>
-  <link name="tool_case_y_minus_x_positive_face"/>
-  <joint name="tool_case_y_minus_to_x_positive_face" type="fixed">
-    <parent link="tool_case_y_minus"/><child link="tool_case_y_minus_x_positive_face"/>
-    <origin xyz="0.0184 0 0" rpy="0 1.570796326795 0"/>
-  </joint>
-  <link name="tool_case_y_minus_x_negative_face"/>
-  <joint name="tool_case_y_minus_to_x_negative_face" type="fixed">
-    <parent link="tool_case_y_minus"/><child link="tool_case_y_minus_x_negative_face"/>
-    <origin xyz="-0.0184 0 0" rpy="0 -1.570796326795 0"/>
+  <!-- Former case 3 location: supply-box pickup area, not a measured grasp pose.
+       No permanent collision; reference axes are parallel to world. -->
+  <link name="supplybox_pickup_area"/>
+  <joint name="arm_world_to_supplybox_pickup_area" type="fixed">
+    <parent link="arm_world"/><child link="supplybox_pickup_area"/>
+    <origin xyz="-0.268 -0.10245 0.153595589" rpy="0 0 0"/>
   </joint>
   <!-- Tool case 1: outer 36.8(X) x 100(Y) x 80(Z) mm.

File: src/arm/tool_manipulator_moveit_config/config/tool_manipulator.ros2_control.xacro (robot description, xacro)
@@ -90,5 +90,5 @@
           <param name="port_name">${hw['buses']['dynamixel_u2d2']['device']}</param>
           <param name="baud_rate">${hw['buses']['dynamixel_u2d2']['baud_rate']}</param>
-          <param name="u2d2_mixed_ttl_rs485">${hw['buses']['dynamixel_u2d2']['mixed_ttl_rs485']}</param>
+          <param name="u2d2_mixed_ttl_rs485">${'true' if hw['buses']['dynamixel_u2d2']['mixed_ttl_rs485'] else 'false'}</param>
           <param name="feedback_mode">${hw['buses']['dynamixel_u2d2']['feedback_mode']}</param>
           <param name="command_mode">${hw['buses']['dynamixel_u2d2']['command_mode']}</param>

Commit message: 수동 조작(각 관절별-teleop_sep.py/숙이기 일체형 둘 다-teleop.py) 수정 및 추가 & 툴 교체 박스 정중앙 좌표 수정

File: src/arm/tool_manipulator_description/urdf/tool_manipulator.urdf.xacro (robot description, xacro)
@@ -172,6 +172,8 @@
   <joint name="arm_world_to_tool_case_1" type="fixed">
     <parent link="arm_world"/><child link="tool_case_1"/>
+    <!-- Gripper-case centre measured from the base axis: X=-394.506, Z=212.964 mm.
+         base_actuator and arm_world share the same origin and orientation. -->
     <!-- arm_world has world orientation, so pitch +55 deg is world-Y tilt. -->
-    <origin xyz="-0.427272082 0 0.190020943" rpy="0 0.959931088597 0"/>
+    <origin xyz="-0.394506 0 0.212964" rpy="0 0.959931088597 0"/>
   </joint>
   <!-- Case-1 local YZ outer faces, at X = +/-18.4 mm. The positive face is the EE entry. -->

Commit message: 다이나믹셀 허브 문제 해결1

File: src/arm/tool_manipulator_description/urdf/tool_manipulator.urdf.xacro (robot description, xacro)
@@ -481,9 +481,8 @@
        the same physical output shaft rather than declaring its own motor joint. -->
   <link name="ee_output_link"/>
-  <joint name="ee_joint" type="revolute">
+  <joint name="ee_joint" type="continuous">
     <parent link="tcp_link"/><child link="ee_output_link"/>
     <origin xyz="0 0 0" rpy="0 0 0"/><axis xyz="0 0 1"/>
-    <!-- raw 1992 = 0 rad; raw 459..3843 are the measured safe endpoints. -->
-    <limit lower="-2.351592547829" upper="2.839398438376" effort="8.4" velocity="5.035177"/>
+    <limit effort="8.4" velocity="5.035177"/>
   </joint>
   <!-- RealSense D435 bracket: TCP is the mechanical parent frame. -->

File: src/arm/tool_manipulator_moveit_config/config/tool_manipulator.ros2_control.xacro (robot description, xacro)
@@ -43,8 +43,16 @@
   <xacro:macro name="dxl_joint" params="name spec wrap">
     <joint name="${name}">
-      <command_interface name="position">
-        <param name="min">${spec['soft_limit_rad'][0]}</param>
-        <param name="max">${spec['soft_limit_rad'][1]}</param>
-      </command_interface>
+      <xacro:if value="${spec['operating_mode'] == 1}">
+        <command_interface name="velocity">
+          <param name="min">${-spec['velocity_limit_rad_s']}</param>
+          <param name="max">${spec['velocity_limit_rad_s']}</param>
+        </command_interface>
+      </xacro:if>
+      <xacro:unless value="${spec['operating_mode'] == 1}">
+        <command_interface name="position">
+          <param name="min">${spec['soft_limit_rad'][0]}</param>
+          <param name="max">${spec['soft_limit_rad'][1]}</param>
+        </command_interface>
+      </xacro:unless>
       <state_interface name="position"/><state_interface name="velocity"/><state_interface name="effort"/>
       <!-- Model coordinate is raw_tick*2pi/4096-pi. -->
@@ -58,5 +66,10 @@
       <param name="type">dxl</param><param name="ID">${spec['id']}</param>
       <param name="transport_channel">${spec['transport_channel']}</param>
-      <command_interface name="Goal Position"/>
+      <xacro:if value="${spec['operating_mode'] == 1}">
+        <command_interface name="Goal Velocity"/>
+      </xacro:if>
+      <xacro:unless value="${spec['operating_mode'] == 1}">
+        <command_interface name="Goal Position"/>
+      </xacro:unless>
       <state_interface name="Present Position"/><state_interface name="Present Velocity"/><state_interface name="Present Current"/>
       <param name="Operating Mode">${spec['operating_mode']}</param>

Commit message: Refactor tool management and update tool descriptions
- Removed ToolAttachmentManager and ToolChangeStateMachine scripts as they are no longer needed.
- Updated tool ID descriptions in launch files for clarity on tool types.
- Added new collision and visual mesh files for the tool manipulator.
- Adjusted URDF parameters for the tool manipulator, including TCP offsets and joint limits.
- Modified tool gripper Xacro file to reflect changes in TCP offset and gear specifications.
- Updated demo launch file to align with new tool descriptions.

File: src/arm/tool_manipulator_description/urdf/tool_manipulator.urdf.xacro (robot description, xacro)
@@ -221,6 +221,6 @@
     <!-- 임시 limit -->
     <limit
-        lower="-3.503612119531"
-        upper="3.614058736259"
+        lower="-3.503"
+        upper="3.614"
         effort="1.0"
         velocity="1.0"/>
@@ -264,6 +264,6 @@
     <axis xyz="0 0 -1"/>
     <limit
-        lower="-1.592612942445"
-        upper="1.518069930092"
+        lower="-1.592"
+        upper="1.518"
         effort="1.0"
         velocity="1.0"/>
@@ -307,6 +307,6 @@
     <axis xyz="0 0 -1"/>
     <limit
-        lower="-1.497824110769"
-        upper="1.542679072545"
+        lower="-1.497"
+        upper="1.542"
         effort="1.0"
         velocity="1.0"/>
@@ -350,6 +350,6 @@
     <axis xyz="0 0 -1"/>
     <limit
-        lower="-1.592420956227"
-        upper="1.470596974438"
+        lower="-1.592"
+        upper="1.470"
         effort="1.0"
         velocity="1.0"/>
@@ -442,9 +442,11 @@
   </joint>
   <!-- ========================================================= -->
-  <!-- EE ACTUATOR -->
-  <!-- wrist yaw -> EE hinge/TCP = +62 mm world Z -->
+  <!-- EE ACTUATOR DRIVE GEAR -->
+  <!-- wrist yaw -> EE drive gear centre:
+       wrist-yaw local (-34, 0, +78.36) mm
+       measured world (0, -34, +78.36) mm -->
   <!-- wrist_yaw frame -->
-  <!-- Xe = -Yworld -->
-  <!-- Ye = +Xworld -->
+  <!-- Xe = +Yworld -->
+  <!-- Ye = -Xworld -->
   <!-- Ze = +Zworld -->
   <!-- 따라서 local displacement = (0,0,+62 mm) -->
@@ -452,5 +454,5 @@
   <link name="ee_actuator">
     <xacro:mesh_visual
-        mesh="ee_actuator"
+        mesh="ee_gear"
         material="motor_grey"/>
   </link>
@@ -460,19 +462,19 @@
     <child link="ee_actuator"/>
     <origin
-        xyz="0 0 0.062000"
-        rpy="0 0 ${pi/2}"/>
+        xyz="-0.034000 0 0.078360"
+        rpy="0 0 0"/>
   </joint>
   <!-- ========================================================= -->
   <!-- TCP -->
-  <!-- EE actuator hinge center 자체가 TCP -->
-  <!-- 따라서 추가 62 mm를 절대 넣지 않음 -->
+  <!-- Driven tool spur-gear centre is the common TCP.  It is a sibling of
+       ee_actuator because the drive-gear centre is offset by 34 mm. -->
   <!-- ========================================================= -->
   <link name="tcp_link"/>
   <joint name="tcp_joint"
          type="fixed">
-    <parent link="ee_actuator"/>
+    <parent link="wrist_link_yaw"/>
     <child link="tcp_link"/>
     <origin
-        xyz="0 0 0"
+        xyz="0 0 0.078360"
         rpy="0 0 0"/>
   </joint>
@@ -486,5 +488,7 @@
     <limit effort="8.4" velocity="5.035177"/>
   </joint>
-  <!-- RealSense D435 bracket: TCP is the mechanical parent frame. -->
+  <!-- RealSense D435 bracket, measured from TCP in world axes at zero pose:
+       world X=-86.394 mm, Z=-18.9 mm.  In the wrist-yaw/TCP frame,
+       local +Y is world -X and local +Z is world +Z. -->
   <link name="cam_link">
     <xacro:mesh_visual
@@ -494,18 +498,18 @@
   <joint name="cam_link_mount"
          type="fixed">
-    <parent link="wrist_link_yaw"/>
+    <parent link="tcp_link"/>
     <child link="cam_link"/>
     <origin
-        xyz="0 0.0607680 0.074000"
+        xyz="0 0.086394 -0.018900"
         rpy="${-pi/2} ${-pi/2} 0"/>
   </joint>
   <!-- The common arm ends at tcp_link; the selected tool is downstream. -->
-  <xacro:if value="${selected_tool_id == 1}">
+  <xacro:if value="${selected_tool_id == 0}">
     <xacro:tool_1_gripper prefix="" parent="ee_output_link" use_mesh="$(arg use_mesh)"/>
   </xacro:if>
-  <xacro:if value="${selected_tool_id == 2}">
+  <xacro:if value="${selected_tool_id == 1}">
     <xacro:tool_2 prefix="" parent="ee_output_link" use_mesh="$(arg use_mesh)"/>
   </xacro:if>
-  <xacro:if value="${selected_tool_id == 3}">
+  <xacro:if value="${selected_tool_id == 2}">
     <xacro:tool_3 prefix="" parent="ee_output_link" use_mesh="$(arg use_mesh)"/>
   </xacro:if>

File: src/arm/tool_manipulator_description/urdf/tools/tool_1_gripper.xacro (robot description, xacro)
@@ -4,5 +4,5 @@
 <robot xmlns:xacro="http://www.ros.org/wiki/xacro">
   <xacro:macro name="tool_1_gripper" params="prefix parent use_mesh:=false">
-    <xacro:property name="tool_1_tcp_offset" value="0.090"/>
+    <xacro:property name="tool_1_tcp_offset" value="0.0256"/>
     <!-- MX-106 raw reference: raw 1992 = 0 rad; raw increment = CCW/closing; 4096 tick/rev. -->
     <xacro:property name="tool_1_gripper_limit_lower" value="-2.351592547829"/> <!-- raw 459 -->
@@ -25,21 +25,20 @@
     </joint>
     <link name="${prefix}tool_1_geometry_link"/>
-    <!-- ========== ee_joint output -> pinion_gear (revolute, "피니언 구동") ==========-->
-    <joint name="pinion_gear_mount_joint" type="fixed">
-      <parent link="tool_1_geometry_link"/>
-      <child link="pinion_gear"/>
-      <origin xyz="0 0 0" rpy="0 -e 0"/>
+    <!-- The gripper's driven spur gear is concentric with tcp_link/ee_joint. -->
+    <joint name="${prefix}tool_spurgear_mount_joint" type="fixed">
+      <parent link="${prefix}tool_1_link"/>
+      <child link="${prefix}tool_spurgear"/>
+      <origin xyz="0 0 0" rpy="0 0 0"/>
     </joint>
-    <!-- pinion_gear: m=1, z=34, 피치반경 17mm (module 1 x teeth 34 / 2, 2026-08-30 mesh 개정) -->
-    <link name="${prefix}pinion_gear">
+    <link name="${prefix}tool_spurgear">
       <xacro:if value="${use_mesh}">
         <visual>
           <origin xyz="0 0 0" rpy="0 0 0"/>
-          <geometry><mesh filename="package://tool_manipulator_description/meshes/visual/pinion_gear.stl" scale="0.001 0.001 0.001"/></geometry>
+          <geometry><mesh filename="package://tool_manipulator_description/meshes/visual/tool_spurgear.stl" scale="0.001 0.001 0.001"/></geometry>
           <material name="motor_dark"/>
         </visual>
         <collision>
           <origin xyz="0 0 0" rpy="0 0 0"/>
-          <geometry><mesh filename="package://tool_manipulator_description/meshes/collision/pinion_gear.stl" scale="0.001 0.001 0.001"/></geometry>
+          <geometry><mesh filename="package://tool_manipulator_description/meshes/collision/tool_spurgear.stl" scale="0.001 0.001 0.001"/></geometry>
         </collision>
       </xacro:if>
@@ -47,10 +46,10 @@
         <visual>
           <origin xyz="0 0 0" rpy="0 0 0"/>
-          <geometry><cylinder radius="0.016" length="0.012"/></geometry>
+          <geometry><cylinder radius="0.018" length="0.0508"/></geometry>
           <material name="motor_dark"/>
         </visual>
         <collision>
           <origin xyz="0 0 0" rpy="0 0 0"/>
-          <geometry><cylinder radius="0.016" length="0.012"/></geometry>
+          <geometry><cylinder radius="0.018" length="0.0508"/></geometry>
         </collision>
       </xacro:unless>
@@ -61,4 +60,11 @@
       </inertial>
     </link>
+    <!-- Tool 0 working TCP: +25.6 mm along world/local Z from tcp_link. -->
+    <joint name="${prefix}tool_1_tcp_joint" type="fixed">
+      <parent link="${prefix}tool_1_link"/>
+      <child link="${prefix}tool_1_tcp"/>
+      <origin xyz="0 0 ${tool_1_tcp_offset}" rpy="0 0 0"/>
+    </joint>
+    <link name="${prefix}tool_1_tcp"/>
     <!-- ========== wrist_link -> rack_left (prismatic, mimic) ==========-->
     <joint name="${prefix}rack_left_joint" type="prismatic">

Commit message: STL 파일 업데이트 및 URDF에서 메쉬 시각화 매크로 수정

File: src/arm/tool_manipulator_description/urdf/tool_manipulator.urdf.xacro (robot description, xacro)
@@ -48,5 +48,5 @@
   <!-- STL 단위 mm -> URDF m -->
   <!-- ========================================================= -->
-  <xacro:macro name="mesh_visual" params="mesh material">
+  <xacro:macro name="mesh_visual" params="mesh material mesh_rpy:='0 0 0'">
     <xacro:if value="$(arg use_mesh)">
       <visual>
@@ -55,8 +55,8 @@
         STL export origin = 해당 hinge
         STL export axes   = 해당 local frame
-        따라서 여기서 추가 회전/이동 금지.
+        기본적으로 추가 이동은 없으며, CAD 정렬이 필요한 링크만 mesh_rpy를 사용한다.
       -->
       <origin xyz="0 0 0"
-              rpy="0 0 0"/>
+              rpy="${mesh_rpy}"/>
       <geometry>
         <mesh
@@ -67,5 +67,5 @@
     </visual>
       <collision>
-        <origin xyz="0 0 0" rpy="0 0 0"/>
+        <origin xyz="0 0 0" rpy="${mesh_rpy}"/>
         <geometry>
           <mesh filename="${collision_mesh_path}/${mesh}.stl" scale="0.001 0.001 0.001"/>
@@ -296,5 +296,6 @@
     <xacro:mesh_visual
         mesh="elbow_link"
-        material="petg_charcoal"/>
+        material="petg_charcoal"
+        mesh_rpy="0 ${pi} 0"/>
   </link>
   <joint name="elbow_joint"
@@ -444,6 +445,6 @@
   <!-- EE ACTUATOR DRIVE GEAR -->
   <!-- wrist yaw -> EE drive gear centre:
-       wrist-yaw local (-34, 0, +78.36) mm
-       measured world (0, -34, +78.36) mm -->
+       wrist-yaw local (0, +34, +78.36) mm
+       measured world (-34, 0, +78.36) mm -->
   <!-- wrist_yaw frame -->
   <!-- Xe = +Yworld -->
@@ -462,5 +463,5 @@
     <child link="ee_actuator"/>
     <origin
-        xyz="-0.034000 0 0.078360"
+        xyz="0 0.034000 0.078360"
         rpy="0 0 0"/>
   </joint>

File: src/arm/tool_manipulator_description/urdf/tools/tool_1_gripper.xacro (robot description, xacro)
@@ -72,9 +72,8 @@
       <child  link="${prefix}rack_left"/>
       <xacro:property name="pinion_pitch_radius" value="0.017"/>
-      <!-- z: pinion_gear 원점(wrist_link 기준 z=${-off_wrist})에서 +0.062 오프셋.
-           기존에는 wrist_link의 z=0을 중심으로 ±0.062를 줘서 pinion_gear
-           원점(z=${-off_wrist})만큼 어긋나 있었음 - 2026-08-24 수정. -->
-      <origin xyz="-0.016 0.018 0.062" rpy="${pi} 0 ${pi}"/>
+      <!-- TCP-local origin after tool_1_geometry rotation: (0, +62, 0) mm.
+           Both racks share the TCP X coordinate and world-Z height. -->
       <axis xyz="0 0 1"/>
+      <origin xyz="0 0 0.062" rpy="${pi} 0 ${pi}"/>
       <limit lower="0" upper="0.030" effort="8.4" velocity="0.1"/>
       <!-- ee_joint 각속도 -> 랙 선속도 변환: v = omega * pinion_pitch_radius.
@@ -88,13 +87,13 @@
     <link name="${prefix}rack_left">
       <xacro:if value="${use_mesh}">
-        <!-- [시각화] parent/rpy가 새로 바뀌어 기존 mesh 보정값이 더 이상
-             맞지 않음 - 시각적으로 다시 맞춰야 함(우선 무회전으로 둠). -->
+        <!-- +90 deg about world Z at the zero pose.  In rack_left coordinates,
+             world +Z is local +X. -->
         <visual>
-          <origin xyz="0 0 0" rpy="0 0 0"/>
+          <origin xyz="0 0 0" rpy="${pi/2} 0 0"/>
           <geometry><mesh filename="package://tool_manipulator_description/meshes/visual/rack_left.stl" scale="0.001 0.001 0.001"/></geometry>
           <material name="petg_grey"/>
         </visual>
         <collision>
-          <origin xyz="0 0 0" rpy="0 0 0"/>
+          <origin xyz="0 0 0" rpy="${pi/2} 0 0"/>
           <geometry><mesh filename="package://tool_manipulator_description/meshes/collision/rack_left.stl" scale="0.001 0.001 0.001"/></geometry>
         </collision>
@@ -122,7 +121,6 @@
       <parent link="${prefix}tool_1_geometry_link"/>
       <child  link="${prefix}rack_right"/>
-      <!-- z: pinion_gear 원점(wrist_link 기준 z=${-off_wrist})에서 -0.062 오프셋.
-           rack_left_joint와 동일한 수정 - 2026-08-24. -->
-      <origin xyz="-0.016 -0.018 -0.062" rpy="0 0 0"/>
+      <!-- TCP-local origin after tool_1_geometry rotation: (0, -62, 0) mm. -->
+      <origin xyz="0 0 -0.062" rpy="0 0 0"/>
       <axis xyz="0 0 1"/>
       <limit lower="0" upper="0.030" effort="8.4" velocity="0.1"/>
@@ -132,13 +130,13 @@
     <link name="${prefix}rack_right">
       <xacro:if value="${use_mesh}">
-        <!-- [시각화] parent/rpy가 새로 바뀌어 기존 mesh 보정값이 더 이상
-             맞지 않음 - 시각적으로 다시 맞춰야 함(우선 무회전으로 둠). -->
+        <!-- +90 deg about world Z at the zero pose.  In rack_right coordinates,
+             world +Z is local -X. -->
         <visual>
-          <origin xyz="0 0 0" rpy="0 0 0"/>
+          <origin xyz="0 0 0" rpy="${-pi/2} 0 0"/>
           <geometry><mesh filename="package://tool_manipulator_description/meshes/visual/rack_right.stl" scale="0.001 0.001 0.001"/></geometry>
           <material name="petg_grey"/>
         </visual>
         <collision>
-          <origin xyz="0 0 0" rpy="0 0 0"/>
+          <origin xyz="0 0 0" rpy="${-pi/2} 0 0"/>
           <geometry><mesh filename="package://tool_manipulator_description/meshes/collision/rack_right.stl" scale="0.001 0.001 0.001"/></geometry>
         </collision>
