Commit message: Refactor and clean up tool manipulator codebase
- Removed obsolete test files: test_joint_joy_teleop.py, test_real_control_teleop_launch.py, test_tag1_recorded_path.py, test_tag1_recorded_path_node.py.
- Added new test file: test_real_control_launch.py to inspect core real-control launch without hardware.
- Updated test_manual.py to reflect changes in expected output for joint limits.
- Modified URDF files for tool manipulator and gripper to correct origin and rotation parameters.
- Improved terminal launcher scripts for better workspace handling and command execution.
- Cleaned up bash aliases for manual control to enhance usability.

File: src/arm/tool_manipulator_description/urdf/tool_manipulator.urdf.xacro (robot description, xacro)
@@ -48,5 +48,5 @@
   <!-- STL 단위 mm -> URDF m -->
   <!-- ========================================================= -->
-  <xacro:macro name="mesh_visual" params="mesh material mesh_rpy:='0 0 0'">
+  <xacro:macro name="mesh_visual" params="mesh material">
     <xacro:if value="$(arg use_mesh)">
       <visual>
@@ -55,8 +55,8 @@
         STL export origin = 해당 hinge
         STL export axes   = 해당 local frame
-        기본적으로 추가 이동은 없으며, CAD 정렬이 필요한 링크만 mesh_rpy를 사용한다.
+        따라서 여기서 추가 회전/이동 금지.
       -->
       <origin xyz="0 0 0"
-              rpy="${mesh_rpy}"/>
+              rpy="0 0 0"/>
       <geometry>
         <mesh
@@ -67,5 +67,5 @@
     </visual>
       <collision>
-        <origin xyz="0 0 0" rpy="${mesh_rpy}"/>
+        <origin xyz="0 0 0" rpy="0 0 0"/>
         <geometry>
           <mesh filename="${collision_mesh_path}/${mesh}.stl" scale="0.001 0.001 0.001"/>
@@ -296,6 +296,5 @@
     <xacro:mesh_visual
         mesh="elbow_link"
-        material="petg_charcoal"
-        mesh_rpy="0 ${pi} 0"/>
+        material="petg_charcoal"/>
   </link>
   <joint name="elbow_joint"
@@ -305,5 +304,5 @@
     <origin
         xyz="0 0.180000 -0.052578"
-        rpy="${pi} 0 0"/>
+        rpy="0 0 ${pi}"/>
     <axis xyz="0 0 -1"/>
     <limit
@@ -434,5 +433,5 @@
     <origin
         xyz="-0.075000 0 0"
-        rpy="${pi/2} 0 ${-pi/2}"/>
+        rpy="${-pi/2} 0 ${pi/2}"/>
     <axis xyz="0 0 1"/>
     <limit
@@ -489,7 +488,7 @@
     <limit effort="8.4" velocity="5.035177"/>
   </joint>
-  <!-- RealSense D435 bracket, measured from TCP in world axes at zero pose:
-       world X=-86.394 mm, Z=-18.9 mm.  In the wrist-yaw/TCP frame,
-       local +Y is world -X and local +Z is world +Z. -->
+  <!-- RealSense D435 origin in the wrist-yaw frame:
+       (X=0, Y=+94.768, Z=+59.46) mm.  Since tcp_link is at wrist-yaw
+       Z=+78.36 mm with the same orientation, the TCP-relative Z is -18.9 mm. -->
   <link name="cam_link">
     <xacro:mesh_visual
@@ -502,5 +501,5 @@
     <child link="cam_link"/>
     <origin
-        xyz="0 0.086394 -0.018900"
+        xyz="0 0.094768 -0.018900"
         rpy="${-pi/2} ${-pi/2} 0"/>
   </joint>

File: src/arm/tool_manipulator_description/urdf/tools/tool_1_gripper.xacro (robot description, xacro)
@@ -72,8 +72,10 @@
       <child  link="${prefix}rack_left"/>
       <xacro:property name="pinion_pitch_radius" value="0.017"/>
-      <!-- TCP-local origin after tool_1_geometry rotation: (0, +62, 0) mm.
-           Both racks share the TCP X coordinate and world-Z height. -->
+      <!-- rack_left origin from wrist_yaw in world axes:
+           (X=+34, Y=-62, Z=+78.36) mm.
+           URDF xyz below is expressed in tool_1_geometry_link.
+           The joint rpy also carries the requested world-Z +90 deg rotation. -->
       <axis xyz="0 0 1"/>
-      <origin xyz="0 0 0.062" rpy="${pi} 0 ${pi}"/>
+      <origin xyz="0 0.062 -0.034" rpy="${-pi/2} 0 ${pi}"/>
       <limit lower="0" upper="0.030" effort="8.4" velocity="0.1"/>
       <!-- ee_joint 각속도 -> 랙 선속도 변환: v = omega * pinion_pitch_radius.
@@ -87,13 +89,11 @@
     <link name="${prefix}rack_left">
       <xacro:if value="${use_mesh}">
-        <!-- +90 deg about world Z at the zero pose.  In rack_left coordinates,
-             world +Z is local +X. -->
         <visual>
-          <origin xyz="0 0 0" rpy="${pi/2} 0 0"/>
+          <origin xyz="0 0 0" rpy="0 0 0"/>
           <geometry><mesh filename="package://tool_manipulator_description/meshes/visual/rack_left.stl" scale="0.001 0.001 0.001"/></geometry>
           <material name="petg_grey"/>
         </visual>
         <collision>
-          <origin xyz="0 0 0" rpy="${pi/2} 0 0"/>
+          <origin xyz="0 0 0" rpy="0 0 0"/>
           <geometry><mesh filename="package://tool_manipulator_description/meshes/collision/rack_left.stl" scale="0.001 0.001 0.001"/></geometry>
         </collision>
@@ -121,6 +121,9 @@
       <parent link="${prefix}tool_1_geometry_link"/>
       <child  link="${prefix}rack_right"/>
-      <!-- TCP-local origin after tool_1_geometry rotation: (0, -62, 0) mm. -->
-      <origin xyz="0 0 -0.062" rpy="0 0 0"/>
+      <!-- rack_right origin from wrist_yaw in world axes:
+           (X=-34, Y=+62, Z=+78.36) mm.
+           URDF xyz below is expressed in tool_1_geometry_link.  The joint rpy carries the
+           requested world-Z +90 deg rotation. -->
+      <origin xyz="0 -0.062 0.034" rpy="${-pi/2} 0 0"/>
       <axis xyz="0 0 1"/>
       <limit lower="0" upper="0.030" effort="8.4" velocity="0.1"/>
@@ -130,13 +133,11 @@
     <link name="${prefix}rack_right">
       <xacro:if value="${use_mesh}">
-        <!-- +90 deg about world Z at the zero pose.  In rack_right coordinates,
-             world +Z is local -X. -->
         <visual>
-          <origin xyz="0 0 0" rpy="${-pi/2} 0 0"/>
+          <origin xyz="0 0 0" rpy="0 0 0"/>
           <geometry><mesh filename="package://tool_manipulator_description/meshes/visual/rack_right.stl" scale="0.001 0.001 0.001"/></geometry>
           <material name="petg_grey"/>
         </visual>
         <collision>
-          <origin xyz="0 0 0" rpy="${-pi/2} 0 0"/>
+          <origin xyz="0 0 0" rpy="0 0 0"/>
           <geometry><mesh filename="package://tool_manipulator_description/meshes/collision/rack_right.stl" scale="0.001 0.001 0.001"/></geometry>
         </collision>

Commit message: test: Add regression test for measured stop pose in camera world height fix: Update home joint values to match manual.py STOP_POSE_RAD

File: src/arm/tool_manipulator_description/urdf/tool_manipulator.urdf.xacro (robot description, xacro)
@@ -48,5 +48,5 @@
   <!-- STL 단위 mm -> URDF m -->
   <!-- ========================================================= -->
-  <xacro:macro name="mesh_visual" params="mesh material">
+  <xacro:macro name="mesh_visual" params="mesh material mesh_rpy:='0 0 0'">
     <xacro:if value="$(arg use_mesh)">
       <visual>
@@ -55,8 +55,10 @@
         STL export origin = 해당 hinge
         STL export axes   = 해당 local frame
-        따라서 여기서 추가 회전/이동 금지.
+        기본적으로 추가 이동은 없으며, CAD 정렬이 필요한 링크만
+        mesh_rpy로 시각/충돌 형상을 보정한다. 관절 운동학 프레임은
+        메쉬 정렬을 위해 변경하지 않는다.
       -->
       <origin xyz="0 0 0"
-              rpy="0 0 0"/>
+              rpy="${mesh_rpy}"/>
       <geometry>
         <mesh
@@ -67,5 +69,5 @@
     </visual>
       <collision>
-        <origin xyz="0 0 0" rpy="0 0 0"/>
+        <origin xyz="0 0 0" rpy="${mesh_rpy}"/>
         <geometry>
           <mesh filename="${collision_mesh_path}/${mesh}.stl" scale="0.001 0.001 0.001"/>
@@ -296,5 +298,6 @@
     <xacro:mesh_visual
         mesh="elbow_link"
-        material="petg_charcoal"/>
+        material="petg_charcoal"
+        mesh_rpy="0 ${pi} 0"/>
   </link>
   <joint name="elbow_joint"
@@ -304,5 +307,5 @@
     <origin
         xyz="0 0.180000 -0.052578"
-        rpy="0 0 ${pi}"/>
+        rpy="${pi} 0 0"/>
     <axis xyz="0 0 -1"/>
     <limit
@@ -433,5 +436,5 @@
     <origin
         xyz="-0.075000 0 0"
-        rpy="${-pi/2} 0 ${pi/2}"/>
+        rpy="${pi/2} 0 ${-pi/2}"/>
     <axis xyz="0 0 1"/>
     <limit
@@ -444,5 +447,5 @@
   <!-- EE ACTUATOR DRIVE GEAR -->
   <!-- wrist yaw -> EE drive gear centre:
-       wrist-yaw local (0, +34, +78.36) mm
+       wrist-yaw local (0, -34, +78.36) mm
        measured world (-34, 0, +78.36) mm -->
   <!-- wrist_yaw frame -->
@@ -462,5 +465,5 @@
     <child link="ee_actuator"/>
     <origin
-        xyz="0 0.034000 0.078360"
+        xyz="0 -0.034000 0.078360"
         rpy="0 0 0"/>
   </joint>

Commit message: 하하~

File: src/arm/tool_manipulator_description/urdf/tool_manipulator.urdf.xacro (robot description, xacro)
@@ -18,4 +18,11 @@
   <xacro:arg name="arm_world_z" default="0.235"/>
   <xacro:arg name="imu_height_from_ground" default="0.115"/>
+  <!-- D435 mounting-centre -> depth/base origin, in the camera body axes
+       X forward, Y left, Z up.  Nominal values follow the official D435
+       description: 14.9 - 0.1 - 4.2 = 10.6 mm forward, 17.5 mm left,
+       and half the 25 mm enclosure height. -->
+  <xacro:arg name="camera_depth_from_mount_x" default="0.0106"/>
+  <xacro:arg name="camera_depth_from_mount_y" default="0.0175"/>
+  <xacro:arg name="camera_depth_from_mount_z" default="0.0125"/>
   <xacro:include filename="tools/tool_1_gripper.xacro"/>
   <xacro:property name="selected_tool_id" value="$(arg tool_id)"/>
@@ -491,7 +498,8 @@
     <limit effort="8.4" velocity="5.035177"/>
   </joint>
-  <!-- RealSense D435 origin in the wrist-yaw frame:
+  <!-- Physical D435 mounting/bolt centre in the wrist-yaw frame:
        (X=0, Y=+94.768, Z=+59.46) mm.  Since tcp_link is at wrist-yaw
-       Z=+78.36 mm with the same orientation, the TCP-relative Z is -18.9 mm. -->
+       Z=+78.36 mm with the same orientation, the TCP-relative Z is -18.9 mm.
+       cam_link axes are X forward, Y left, Z up. -->
   <link name="cam_link">
     <xacro:mesh_visual
@@ -506,4 +514,14 @@
         xyz="0 0.094768 -0.018900"
         rpy="${-pi/2} ${-pi/2} 0"/>
+  </joint>
+  <!-- realsense2_camera prefixes camera_name=arm_camera to base_frame_id,
+       producing arm_camera_cam_link.  The driver uses that root as the depth
+       sensor origin, so it is offset from the physical mounting centre. -->
+  <link name="arm_camera_cam_link"/>
+  <joint name="cam_link_to_realsense_base" type="fixed">
+    <parent link="cam_link"/>
+    <child link="arm_camera_cam_link"/>
+    <origin xyz="$(arg camera_depth_from_mount_x) $(arg camera_depth_from_mount_y) $(arg camera_depth_from_mount_z)"
+            rpy="0 0 0"/>
   </joint>
   <!-- The common arm ends at tcp_link; the selected tool is downstream. -->

Commit message: 회로박스 충돌박스 urdf에 반영

File: src/arm/tool_manipulator_description/urdf/tool_manipulator.urdf.xacro (robot description, xacro)
@@ -18,4 +18,10 @@
   <xacro:arg name="arm_world_z" default="0.235"/>
   <xacro:arg name="imu_height_from_ground" default="0.115"/>
+  <!-- Wheel radius in rmd_x8_params.yaml; with the wheel on the ground,
+       its axle centre is this height above ground. -->
+  <xacro:arg name="wheel_axle_height_from_ground" default="0.1125"/>
+  <xacro:property name="wheel_axle_z" value="$(arg wheel_axle_height_from_ground)"/>
+  <xacro:property name="imu_z" value="$(arg imu_height_from_ground)"/>
+  <xacro:property name="chassis_mount_z_m" value="$(arg chassis_mount_z)"/>
   <!-- D435 mounting-centre -> depth/base origin, in the camera body axes
        X forward, Y left, Z up.  Nominal values follow the official D435
@@ -104,14 +110,28 @@
     <origin xyz="$(arg chassis_mount_x) $(arg chassis_mount_y) $(arg chassis_mount_z)" rpy="0 0 0"/>
   </joint>
-  <!-- Circuit-box centre in base_actuator coordinates:
-       (-161.6 - 28 - 170, 0, 36) mm = (-359.6, 0, 36) mm.
-       Top is 137 + 300 = 437 mm above ground; box height 102 mm gives centre z=386 mm ground, or 36 mm from base. -->
+  <!-- Circuit-box footprint from the eight measured points, in millimetres
+       relative to the chassis centre: CAD X points right and CAD Y points
+       forward. URDF X points forward and URDF Y points left, so
+       (X_URDF, Y_URDF) = (Y_CAD, -X_CAD).
+       The points specify the top at wheel-axle-centre Z=372 mm. Keep the
+       previous 102 mm box height until a bottom-face measurement is available.
+       The three boxes fill the rear bar and side arms, leaving the central
+       140 x 120 mm opening empty. -->
   <link name="circuit_box">
-    <visual><geometry><box size="0.340 0.280 0.102"/></geometry><material name="circuit_box_orange"/></visual>
-    <collision><geometry><box size="0.340 0.280 0.102"/></geometry></collision>
-  </link>
-  <joint name="base_actuator_to_circuit_box" type="fixed">
-    <parent link="base_actuator"/><child link="circuit_box"/>
-    <origin xyz="-0.3596 0 0.036" rpy="0 0 0"/>
+    <!-- CAD X +/-170, Y -274.097..-114.097 mm: rear bar. -->
+    <visual><origin xyz="-0.060 0 0"/><geometry><box size="0.160 0.340 0.102"/></geometry><material name="circuit_box_orange"/></visual>
+    <collision><origin xyz="-0.060 0 0"/><geometry><box size="0.160 0.340 0.102"/></geometry></collision>
+    <!-- CAD X -170..-70, Y -114.097..5.903 mm: left side. -->
+    <visual><origin xyz="0.080 0.120 0"/><geometry><box size="0.120 0.100 0.102"/></geometry><material name="circuit_box_orange"/></visual>
+    <collision><origin xyz="0.080 0.120 0"/><geometry><box size="0.120 0.100 0.102"/></geometry></collision>
+    <!-- CAD X 70..170, Y -114.097..5.903 mm: right side. -->
+    <visual><origin xyz="0.080 -0.120 0"/><geometry><box size="0.120 0.100 0.102"/></geometry><material name="circuit_box_orange"/></visual>
+    <collision><origin xyz="0.080 -0.120 0"/><geometry><box size="0.120 0.100 0.102"/></geometry></collision>
+  </link>
+  <joint name="chassis_to_circuit_box" type="fixed">
+    <parent link="chassis"/><child link="circuit_box"/>
+    <!-- X/Y use the chassis centre. Z uses the wheel axle: box centre is
+         axle height + (372 - 102/2) mm, then converted to chassis Z. -->
+    <origin xyz="-0.134097 0 ${float(wheel_axle_z) + 0.321 - float(imu_z) - float(chassis_mount_z_m)}" rpy="0 0 0"/>
   </joint>
   <!-- Robot-arm reference: base height is 350 mm above ground, therefore 235 mm above the IMU/world at ground z=115 mm. -->

Commit message: urdf 그리퍼 핑거 좌표 수정

File: src/arm/tool_manipulator_description/urdf/tool_manipulator.urdf.xacro (robot description, xacro)
@@ -152,12 +152,12 @@
     <collision><origin xyz="0.0104 0.0157 0"/><geometry><box size="0.016 0.0154 0.050"/></geometry></collision>
   </xacro:macro>
-  <!-- Case 2 (+Y) centre is an arm_world offset. Its Z
-       centre is calibrated so the tilted local +Z outer-face midpoint is
-       z=167.935 mm in arm_world. -->
+  <!-- Case 2 (+Y) centre is an arm_world offset. With the 55-degree tilt,
+       the lowest corner of its collision geometry meets the circuit-box top
+       at world Z=369.5 mm for the default mounting dimensions. -->
   <link name="tool_case_y_plus"><xacro:tool_case_walls/></link>
   <joint name="arm_world_to_tool_case_y_plus" type="fixed">
     <parent link="arm_world"/><child link="tool_case_y_plus"/>
     <!-- arm_world has world orientation, so pitch +55 deg is world-Y tilt. -->
-    <origin xyz="-0.268 0.10245 0.153595589" rpy="0 0.959931088597 0"/>
+    <origin xyz="-0.268 0.10245 0.163911809" rpy="0 0.959931088597 0"/>
   </joint>
   <!-- Each dock face is the case local YZ plane at outer X = +/-18.4 mm.
@@ -510,6 +510,6 @@
   </joint>
   <!-- Common end-effector output: Dynamixel ID 4 is always ee_joint.
-       Tools mount downstream of ee_output_link, so each selected tool shares
-       the same physical output shaft rather than declaring its own motor joint. -->
+       Tool 1 fixes its housing and racks to tcp_link and mounts only the driven
+       spur gear on ee_output_link. Other tools use the rotating output. -->
   <link name="ee_output_link"/>
   <joint name="ee_joint" type="continuous">
@@ -547,5 +547,5 @@
   <!-- The common arm ends at tcp_link; the selected tool is downstream. -->
   <xacro:if value="${selected_tool_id == 0}">
-    <xacro:tool_1_gripper prefix="" parent="ee_output_link" use_mesh="$(arg use_mesh)"/>
+    <xacro:tool_1_gripper prefix="" parent="tcp_link" drive_parent="ee_output_link" use_mesh="$(arg use_mesh)"/>
   </xacro:if>
   <xacro:if value="${selected_tool_id == 1}">

File: src/arm/tool_manipulator_description/urdf/tools/tool_1_gripper.xacro (robot description, xacro)
@@ -1,7 +1,7 @@
 <?xml version="1.0"?>
-<!-- Tool 1: existing MX-106T gripper, pinion and racks.  This file owns every
-     link downstream of the common tcp_link; it is never part of no-tool URDF. -->
+<!-- Tool 1: existing MX-106T gripper, pinion and racks. The housing and racks
+     attach to tcp_link; only the pinion attaches to the rotating ee output. -->
 <robot xmlns:xacro="http://www.ros.org/wiki/xacro">
-  <xacro:macro name="tool_1_gripper" params="prefix parent use_mesh:=false">
+  <xacro:macro name="tool_1_gripper" params="prefix parent drive_parent use_mesh:=false">
     <xacro:property name="tool_1_tcp_offset" value="0.0256"/>
     <!-- MX-106 raw reference: raw 1992 = 0 rad; raw increment = CCW/closing; 4096 tick/rev. -->
@@ -10,5 +10,11 @@
     <xacro:property name="tool_1_gripper_close" value="1.251728"/> <!-- measured raw 2808 -->
     <xacro:property name="tool_1_gripper_limit_upper" value="2.839398438376"/> <!-- raw 3843 -->
-    <xacro:property name="tool_1_rack_offset" value="0.018"/>
+    <!-- Rail groove: |TCP Y|=20.8..24.0 mm, TCP Z=21.3..38.9 mm.
+         Rack flange: |TCP Y|=21.0..23.8 mm, TCP Z=21.6..38.6 mm. -->
+    <xacro:property name="tool_1_rack_offset" value="0.01825"/>
+    <xacro:property name="tool_1_rack_height" value="0.0253"/>
+    <!-- Left STL was exported with a -2.821821-degree roll about its slide
+         axis. Undo that mesh tilt to seat its flange parallel to the rail. -->
+    <xacro:property name="tool_1_left_mesh_yaw" value="0.049250067850631254"/>
     <xacro:property name="tool_1_pitch_radius" value="0.017"/>
     <joint name="${prefix}tool_1_mount_joint" type="fixed">
@@ -19,13 +25,13 @@
       <inertial><mass value="0.001"/><inertia ixx="1e-7" ixy="0" ixz="0" iyy="1e-7" iyz="0" izz="1e-7"/></inertial>
     </link>
-    <!-- Common tool geometry frame: from tcp_link, rotate Y +90 deg then Z +90 deg. -->
+    <!-- Rack frame raised to the wrist housing's upper guide slots. -->
     <joint name="${prefix}tool_1_geometry_joint" type="fixed">
       <parent link="${prefix}tool_1_link"/><child link="${prefix}tool_1_geometry_link"/>
-      <origin xyz="0 0 0" rpy="0 ${pi/2} ${pi/2}"/>
+      <origin xyz="0 0 ${tool_1_rack_height}" rpy="0 ${pi/2} ${pi/2}"/>
     </joint>
     <link name="${prefix}tool_1_geometry_link"/>
     <!-- The gripper's driven spur gear is concentric with tcp_link/ee_joint. -->
     <joint name="${prefix}tool_spurgear_mount_joint" type="fixed">
-      <parent link="${prefix}tool_1_link"/>
+      <parent link="${drive_parent}"/>
       <child link="${prefix}tool_spurgear"/>
       <origin xyz="0 0 0" rpy="0 0 0"/>
@@ -72,10 +78,8 @@
       <child  link="${prefix}rack_left"/>
       <xacro:property name="pinion_pitch_radius" value="0.017"/>
-      <!-- rack_left origin from wrist_yaw in world axes:
-           (X=+34, Y=-62, Z=+78.36) mm.
-           URDF xyz below is expressed in tool_1_geometry_link.
-           The joint rpy also carries the requested world-Z +90 deg rotation. -->
+      <!-- In tcp_link, the left rack joint is at X=-62, Y=-18.25, Z=25.3 mm.
+           The origin below is expressed in tool_1_geometry_link. -->
       <axis xyz="0 0 1"/>
-      <origin xyz="0 0.062 -0.034" rpy="${-pi/2} 0 ${pi}"/>
+      <origin xyz="0 0.062 ${-tool_1_rack_offset}" rpy="${-pi/2} 0 ${pi}"/>
       <limit lower="0" upper="0.030" effort="8.4" velocity="0.1"/>
       <!-- ee_joint 각속도 -> 랙 선속도 변환: v = omega * pinion_pitch_radius.
@@ -90,10 +94,10 @@
       <xacro:if value="${use_mesh}">
         <visual>
-          <origin xyz="0 0 0" rpy="0 0 0"/>
+          <origin xyz="0 0 0" rpy="0 0 ${tool_1_left_mesh_yaw}"/>
           <geometry><mesh filename="package://tool_manipulator_description/meshes/visual/rack_left.stl" scale="0.001 0.001 0.001"/></geometry>
           <material name="petg_grey"/>
         </visual>
         <collision>
-          <origin xyz="0 0 0" rpy="0 0 0"/>
+          <origin xyz="0 0 0" rpy="0 0 ${tool_1_left_mesh_yaw}"/>
           <geometry><mesh filename="package://tool_manipulator_description/meshes/collision/rack_left.stl" scale="0.001 0.001 0.001"/></geometry>
         </collision>
@@ -121,9 +125,6 @@
       <parent link="${prefix}tool_1_geometry_link"/>
       <child  link="${prefix}rack_right"/>
-      <!-- rack_right origin from wrist_yaw in world axes:
-           (X=-34, Y=+62, Z=+78.36) mm.
-           URDF xyz below is expressed in tool_1_geometry_link.  The joint rpy carries the
-           requested world-Z +90 deg rotation. -->
-      <origin xyz="0 -0.062 0.034" rpy="${-pi/2} 0 0"/>
+      <!-- In tcp_link, the right rack joint is at X=+62, Y=+18.25, Z=25.3 mm. -->
+      <origin xyz="0 -0.062 ${tool_1_rack_offset}" rpy="${-pi/2} 0 0"/>
       <axis xyz="0 0 1"/>
       <limit lower="0" upper="0.030" effort="8.4" velocity="0.1"/>
