Commit message: 툴박스 중앙 좌표 구형 점으로 변경

File: src/arm/tool_manipulator_description/urdf/tool_manipulator.urdf.xacro (robot description, xacro)
@@ -48,8 +48,7 @@
   <material name="petg_grey"><color rgba="0.40 0.40 0.42 1.0"/></material>
   <material name="motor_dark"><color rgba="0.12 0.12 0.14 1.0"/></material>
-  <material name="tcp_red"><color rgba="0.90 0.05 0.05 1.0"/></material>
+  <material name="tool_case_marker_blue"><color rgba="0.05 0.35 1.0 1.0"/></material>
   <material name="chassis_blue"><color rgba="0.12 0.22 0.34 0.55"/></material>
   <material name="circuit_box_orange"><color rgba="0.85 0.35 0.05 0.80"/></material>
-  <material name="tool_case_blue"><color rgba="0.10 0.45 0.85 0.70"/></material>
   <!-- MOTOR -->
   <material name="motor_grey">
@@ -141,27 +140,27 @@
     <origin xyz="$(arg arm_world_x) $(arg arm_world_y) $(arg arm_world_z)" rpy="0 0 0"/>
   </joint>
-  <!-- Case 2/3 outer: 36.8(X) x 46.8(Y) x 50(Z) mm.
-       EE entry is local +X; cavity is 16(X depth) x 16(Y) x 50(Z) mm. -->
-  <xacro:macro name="tool_case_walls">
-    <!-- back wall and two Y rails: open local +X face toward the EE -->
-    <visual><origin xyz="-0.008 0 0"/><geometry><box size="0.0208 0.0468 0.050"/></geometry><material name="tool_case_blue"/></visual>
-    <collision><origin xyz="-0.008 0 0"/><geometry><box size="0.0208 0.0468 0.050"/></geometry></collision>
-    <visual><origin xyz="0.0104 -0.0157 0"/><geometry><box size="0.016 0.0154 0.050"/></geometry><material name="tool_case_blue"/></visual>
-    <collision><origin xyz="0.0104 -0.0157 0"/><geometry><box size="0.016 0.0154 0.050"/></geometry></collision>
-    <visual><origin xyz="0.0104 0.0157 0"/><geometry><box size="0.016 0.0154 0.050"/></geometry><material name="tool_case_blue"/></visual>
-    <collision><origin xyz="0.0104 0.0157 0"/><geometry><box size="0.016 0.0154 0.050"/></geometry></collision>
+  <!-- Visible centre marker only; it does not affect collision checking. -->
+  <xacro:macro name="tool_case_center_marker" params="case_link marker_link">
+    <link name="${marker_link}">
+      <visual>
+        <origin xyz="0 0 0" rpy="0 0 0"/>
+        <geometry><sphere radius="0.012"/></geometry>
+        <material name="tool_case_marker_blue"/>
+      </visual>
+    </link>
+    <joint name="${case_link}_to_center_marker" type="fixed">
+      <parent link="${case_link}"/><child link="${marker_link}"/>
+      <origin xyz="0 0 0" rpy="0 0 0"/>
+    </joint>
   </xacro:macro>
-  <!-- Case 2 (+Y) centre is an arm_world offset. With the 55-degree tilt,
-       the lowest corner of its collision geometry meets the circuit-box top
-       at world Z=369.5 mm for the default mounting dimensions. -->
-  <link name="tool_case_y_plus"><xacro:tool_case_walls/></link>
+  <!-- Former case 2 frame: +76.7 mm X and +90 mm Y from case 1 in arm_world. -->
+  <link name="tool_case_y_plus"/>
   <joint name="arm_world_to_tool_case_y_plus" type="fixed">
     <parent link="arm_world"/><child link="tool_case_y_plus"/>
-    <!-- arm_world has world orientation, so pitch +55 deg is world-Y tilt. -->
-    <origin xyz="-0.268 0.10245 0.163911809" rpy="0 0.959931088597 0"/>
-  </joint>
-  <!-- Each dock face is the case local YZ plane at outer X = +/-18.4 mm.
-       Its +Z axis is the outward face normal, so an EE TCP XY plane can be
-       made coplanar by aligning TCP +Z with the chosen face normal. -->
+    <!-- Retain the former case-2 orientation for its dock reference frames. -->
+    <origin xyz="-0.317806 0.090 0.163911809" rpy="0 -0.785398163397 0"/>
+  </joint>
+  <xacro:tool_case_center_marker case_link="tool_case_y_plus" marker_link="tool_case_y_plus_center"/>
+  <!-- Former dock reference planes remain at local X = +/-18.4 mm. -->
   <link name="tool_case_y_plus_x_positive_face"/>
   <joint name="tool_case_y_plus_to_x_positive_face" type="fixed">
@@ -181,30 +180,15 @@
     <origin xyz="-0.268 -0.10245 0.153595589" rpy="0 0 0"/>
   </joint>
-  <!-- Tool case 1: outer 36.8(X) x 100(Y) x 80(Z) mm.
-       Entry faces the EE at local +X. Cavity is 16(X depth) x 16(Y) x 50(Z) mm. -->
-  <xacro:macro name="tool_case_1_shell">
-    <!-- back wall: cavity ends 16 mm inboard from local +X entry -->
-    <visual><origin xyz="-0.008 0 0"/><geometry><box size="0.0208 0.100 0.080"/></geometry><material name="tool_case_blue"/></visual>
-    <collision><origin xyz="-0.008 0 0"/><geometry><box size="0.0208 0.100 0.080"/></geometry></collision>
-    <!-- two Y rails around the 16 mm opening -->
-    <visual><origin xyz="0.0104 -0.029 0"/><geometry><box size="0.016 0.042 0.080"/></geometry><material name="tool_case_blue"/></visual>
-    <collision><origin xyz="0.0104 -0.029 0"/><geometry><box size="0.016 0.042 0.080"/></geometry></collision>
-    <visual><origin xyz="0.0104 0.029 0"/><geometry><box size="0.016 0.042 0.080"/></geometry><material name="tool_case_blue"/></visual>
-    <collision><origin xyz="0.0104 0.029 0"/><geometry><box size="0.016 0.042 0.080"/></geometry></collision>
-    <!-- top/bottom rails leave a 50 mm opening along local Z -->
-    <visual><origin xyz="0.0104 0 -0.0325"/><geometry><box size="0.016 0.016 0.015"/></geometry><material name="tool_case_blue"/></visual>
-    <collision><origin xyz="0.0104 0 -0.0325"/><geometry><box size="0.016 0.016 0.015"/></geometry></collision>
-    <visual><origin xyz="0.0104 0 0.0325"/><geometry><box size="0.016 0.016 0.015"/></geometry><material name="tool_case_blue"/></visual>
-    <collision><origin xyz="0.0104 0 0.0325"/><geometry><box size="0.016 0.016 0.015"/></geometry></collision>
-  </xacro:macro>
-  <link name="tool_case_1"><xacro:tool_case_1_shell/></link>
+  <!-- Former case 1 frame retained for its centre marker and dock references. -->
+  <link name="tool_case_1"/>
   <joint name="arm_world_to_tool_case_1" type="fixed">
     <parent link="arm_world"/><child link="tool_case_1"/>
     <!-- Gripper-case centre measured from the base axis: X=-394.506, Z=212.964 mm.
          base_actuator and arm_world share the same origin and orientation. -->
-    <!-- arm_world has world orientation, so pitch +55 deg is world-Y tilt. -->
-    <origin xyz="-0.394506 0 0.212964" rpy="0 0.959931088597 0"/>
-  </joint>
-  <!-- Case-1 local YZ outer faces, at X = +/-18.4 mm. The positive face is the EE entry. -->
+    <!-- Retain the former case-1 orientation for its dock reference frames. -->
+    <origin xyz="-0.394506 0 0.212964" rpy="0 -0.959931088597 0"/>
+  </joint>
+  <xacro:tool_case_center_marker case_link="tool_case_1" marker_link="tool_case_1_center"/>
+  <!-- Former case-1 dock reference planes remain at X = +/-18.4 mm. -->
   <link name="tool_case_1_x_positive_face"/>
   <joint name="tool_case_1_to_x_positive_face" type="fixed">
@@ -291,5 +275,5 @@
         xyz="0 -0.037700 0.103900"
         rpy="${pi/2} 0 0"/>
-    <axis xyz="0 0 -1"/>
+    <axis xyz="0 0 1"/>
     <limit
         lower="-1.592"
@@ -335,5 +319,5 @@
         xyz="0 0.180000 -0.052578"
         rpy="${pi} 0 0"/>
-    <axis xyz="0 0 -1"/>
+    <axis xyz="0 0 1"/>
     <limit
         lower="-1.497"
@@ -378,5 +362,5 @@
         xyz="0 -0.200000 -0.048397"
         rpy="${pi} 0 0"/>
-    <axis xyz="0 0 -1"/>
+    <axis xyz="0 0 1"/>
     <limit
         lower="-1.592"

Commit message: fix: express docking centres in world frame

File: src/arm/tool_manipulator_description/urdf/tool_manipulator.urdf.xacro (robot description, xacro)
@@ -154,10 +154,12 @@
     </joint>
   </xacro:macro>
-  <!-- Former case 2 frame: +76.7 mm X and +90 mm Y from case 1 in arm_world. -->
+  <!-- Tool 1 centre measured in world: (-317.806, +90, +163.912) mm.
+       This joint is expressed in arm_world, whose world offset is
+       (+192.1, 0, +235) mm, hence the converted local origin below. -->
   <link name="tool_case_y_plus"/>
   <joint name="arm_world_to_tool_case_y_plus" type="fixed">
     <parent link="arm_world"/><child link="tool_case_y_plus"/>
     <!-- Retain the former case-2 orientation for its dock reference frames. -->
-    <origin xyz="-0.317806 0.090 0.163911809" rpy="0 -0.785398163397 0"/>
+    <origin xyz="-0.509906 0.090 -0.071088" rpy="0 -0.785398163397 0"/>
   </joint>
   <xacro:tool_case_center_marker case_link="tool_case_y_plus" marker_link="tool_case_y_plus_center"/>
@@ -184,8 +186,9 @@
   <joint name="arm_world_to_tool_case_1" type="fixed">
     <parent link="arm_world"/><child link="tool_case_1"/>
-    <!-- Gripper-case centre measured from the base axis: X=-394.506, Z=212.964 mm.
-         base_actuator and arm_world share the same origin and orientation. -->
+    <!-- Tool 0 centre measured in world: (-394.506, 0, +212.964) mm.
+         Convert to arm_world coordinates by subtracting its
+         (+192.1, 0, +235) mm world offset. -->
     <!-- Retain the former case-1 orientation for its dock reference frames. -->
-    <origin xyz="-0.394506 0 0.212964" rpy="0 -0.959931088597 0"/>
+    <origin xyz="-0.586606 0 -0.022036" rpy="0 -0.959931088597 0"/>
   </joint>
   <xacro:tool_case_center_marker case_link="tool_case_1" marker_link="tool_case_1_center"/>

Commit message: ㅇ

File: src/arm/tool_manipulator_description/urdf/tool_manipulator.urdf.xacro (robot description, xacro)
@@ -154,12 +154,10 @@
     </joint>
   </xacro:macro>
-  <!-- Tool 1 centre measured in world: (-317.806, +90, +163.912) mm.
-       This joint is expressed in arm_world, whose world offset is
-       (+192.1, 0, +235) mm, hence the converted local origin below. -->
+  <!-- Tool 1 centre measured in arm_world: (-317.806, +90, +163.912) mm. -->
   <link name="tool_case_y_plus"/>
   <joint name="arm_world_to_tool_case_y_plus" type="fixed">
     <parent link="arm_world"/><child link="tool_case_y_plus"/>
     <!-- Retain the former case-2 orientation for its dock reference frames. -->
-    <origin xyz="-0.509906 0.090 -0.071088" rpy="0 -0.785398163397 0"/>
+    <origin xyz="-0.317806 0.090 0.163912" rpy="0 -0.785398163397 0"/>
   </joint>
   <xacro:tool_case_center_marker case_link="tool_case_y_plus" marker_link="tool_case_y_plus_center"/>
@@ -186,9 +184,7 @@
   <joint name="arm_world_to_tool_case_1" type="fixed">
     <parent link="arm_world"/><child link="tool_case_1"/>
-    <!-- Tool 0 centre measured in world: (-394.506, 0, +212.964) mm.
-         Convert to arm_world coordinates by subtracting its
-         (+192.1, 0, +235) mm world offset. -->
+    <!-- Tool 0 centre measured in arm_world: (-394.506, 0, +212.964) mm. -->
     <!-- Retain the former case-1 orientation for its dock reference frames. -->
-    <origin xyz="-0.586606 0 -0.022036" rpy="0 -0.959931088597 0"/>
+    <origin xyz="-0.394506 0 0.212964" rpy="0 -0.959931088597 0"/>
   </joint>
   <xacro:tool_case_center_marker case_link="tool_case_1" marker_link="tool_case_1_center"/>

Commit message: 서플라이 박스 추가

File: src/arm/tool_manipulator_description/urdf/tool_manipulator.urdf.xacro (robot description, xacro)
@@ -51,4 +51,5 @@
   <material name="chassis_blue"><color rgba="0.12 0.22 0.34 0.55"/></material>
   <material name="circuit_box_orange"><color rgba="0.85 0.35 0.05 0.80"/></material>
+  <material name="supply_box_green"><color rgba="0.20 0.70 0.30 0.85"/></material>
   <!-- MOTOR -->
   <material name="motor_grey">
@@ -134,4 +135,20 @@
     <origin xyz="-0.134097 0 ${float(wheel_axle_z) + 0.321 - float(imu_z) - float(chassis_mount_z_m)}" rpy="0 0 0"/>
   </joint>
+  <!-- 95 mm supply box on the -Y arm of the U-shaped circuit box, opposite
+       tool case 2. Its bottom rests on the top; its +X face is inset
+       2.5 mm from the protrusion's +X end at local X=0.140 m. -->
+  <link name="supply_box">
+    <visual>
+      <geometry><box size="0.095 0.095 0.095"/></geometry>
+      <material name="supply_box_green"/>
+    </visual>
+    <collision>
+      <geometry><box size="0.095 0.095 0.095"/></geometry>
+    </collision>
+  </link>
+  <joint name="circuit_box_to_supply_box" type="fixed">
+    <parent link="circuit_box"/><child link="supply_box"/>
+    <origin xyz="0.090 -0.120 0.0985" rpy="0 0 0"/>
+  </joint>
   <!-- Robot-arm reference: base height is 350 mm above ground, therefore 235 mm above the IMU/world at ground z=115 mm. -->
   <link name="arm_world"/>
@@ -456,12 +473,6 @@
   <!-- ========================================================= -->
   <!-- EE ACTUATOR DRIVE GEAR -->
-  <!-- wrist yaw -> EE drive gear centre:
-       wrist-yaw local (0, -34, +78.36) mm
-       measured world (-34, 0, +78.36) mm -->
-  <!-- wrist_yaw frame -->
-  <!-- Xe = +Yworld -->
-  <!-- Ye = -Xworld -->
-  <!-- Ze = +Zworld -->
-  <!-- 따라서 local displacement = (0,0,+62 mm) -->
+  <!-- Drive gear sits on the upper side of the gripper housing:
+       wrist-yaw local (0, +34, +78.36) mm. -->
   <!-- ========================================================= -->
   <link name="ee_actuator">

Commit message: ㅇ

File: src/arm/tool_manipulator_description/urdf/tool_manipulator.urdf.xacro (robot description, xacro)
@@ -57,5 +57,6 @@
   </material>
   <!-- ========================================================= -->
-  <!-- VISUAL MACRO -->
+  <!-- VISUAL/COLLISION MACRO. use_mesh controls display only; collision
+       geometry is always present so planning cannot silently become unsafe. -->
   <!-- STL 자체 좌표계를 그대로 사용 -->
   <!-- STL 단위 mm -> URDF m -->
@@ -81,11 +82,23 @@
       <material name="${material}"/>
     </visual>
-      <collision>
+    </xacro:if>
+    <xacro:unless value="$(arg use_mesh)">
+      <!-- Keep RobotModel visible without the detailed visual STL. The
+           collision mesh is reused only for display here; the separate
+           collision element below remains authoritative for planning. -->
+      <visual>
         <origin xyz="0 0 0" rpy="${mesh_rpy}"/>
         <geometry>
           <mesh filename="${collision_mesh_path}/${mesh}.stl" scale="0.001 0.001 0.001"/>
         </geometry>
-      </collision>
-    </xacro:if>
+        <material name="${material}"/>
+      </visual>
+    </xacro:unless>
+    <collision>
+      <origin xyz="0 0 0" rpy="${mesh_rpy}"/>
+      <geometry>
+        <mesh filename="${collision_mesh_path}/${mesh}.stl" scale="0.001 0.001 0.001"/>
+      </geometry>
+    </collision>
   </xacro:macro>
   <!-- ========================================================= -->
@@ -540,5 +553,6 @@
   </joint>
   <!-- The common arm ends at tcp_link; the selected tool is downstream. -->
-  <xacro:if value="${selected_tool_id == 0}">
+  <!-- Supply-box handling (task/tool ID 2) uses the same physical gripper. -->
+  <xacro:if value="${selected_tool_id == 0 or selected_tool_id == 2}">
     <xacro:tool_1_gripper prefix="" parent="tcp_link" drive_parent="ee_output_link" use_mesh="$(arg use_mesh)"/>
   </xacro:if>
@@ -546,6 +560,3 @@
     <xacro:tool_2 prefix="" parent="ee_output_link" use_mesh="$(arg use_mesh)"/>
   </xacro:if>
-  <xacro:if value="${selected_tool_id == 2}">
-    <xacro:tool_3 prefix="" parent="ee_output_link" use_mesh="$(arg use_mesh)"/>
-  </xacro:if>
 </robot>

File: src/arm/tool_manipulator_description/urdf/tools/tool_2.xacro (robot description, xacro)
@@ -2,11 +2,19 @@
 <robot xmlns:xacro="http://www.ros.org/wiki/xacro">
   <xacro:macro name="tool_2" params="prefix parent use_mesh:=false">
-    <joint name="${prefix}tool_2_mount_joint" type="fixed"><parent link="${parent}"/><child link="${prefix}tool_2_link"/><origin xyz="0 0 0.012" rpy="0 0 0"/></joint>
+    <joint name="${prefix}tool_2_mount_joint" type="fixed"><parent link="${parent}"/><child link="${prefix}tool_2_link"/><origin xyz="0 0 0" rpy="0 0 0"/></joint>
     <link name="${prefix}tool_2_link">
-      <visual><geometry><mesh filename="package://tool_manipulator_description/meshes/visual/tool1_drill.stl" scale="0.001 0.001 0.001"/></geometry><material name="motor_grey"/></visual>
+      <xacro:if value="${use_mesh}">
+        <visual><geometry><mesh filename="package://tool_manipulator_description/meshes/visual/tool1_drill.stl" scale="0.001 0.001 0.001"/></geometry><material name="motor_grey"/></visual>
+      </xacro:if>
+      <xacro:unless value="${use_mesh}">
+        <!-- Keep the drill visible in RobotModel while using the lighter
+             collision STL. The fixed parent below makes it rotate 1:1 with
+             ee_output_link/ee_joint. -->
+        <visual><geometry><mesh filename="package://tool_manipulator_description/meshes/collision/tool1_drill.stl" scale="0.001 0.001 0.001"/></geometry><material name="motor_grey"/></visual>
+      </xacro:unless>
       <collision><geometry><mesh filename="package://tool_manipulator_description/meshes/collision/tool1_drill.stl" scale="0.001 0.001 0.001"/></geometry></collision>
-      <inertial><origin xyz="0 0.030 0"/><mass value="0.050"/><inertia ixx="0.00002" ixy="0" ixz="0" iyy="0.000004" iyz="0" izz="0.00002"/></inertial>
+      <inertial><origin xyz="0 0 0.030"/><mass value="0.050"/><inertia ixx="0.00002" ixy="0" ixz="0" iyy="0.00002" iyz="0" izz="0.000004"/></inertial>
     </link>
-    <joint name="${prefix}tool_2_tcp_joint" type="fixed"><parent link="${prefix}tool_2_link"/><child link="${prefix}tool_2_tcp"/><origin xyz="0 0.060 0"/></joint>
+    <joint name="${prefix}tool_2_tcp_joint" type="fixed"><parent link="${prefix}tool_2_link"/><child link="${prefix}tool_2_tcp"/><origin xyz="0 0 0.060"/></joint>
     <link name="${prefix}tool_2_tcp"/>
   </xacro:macro>

File: src/arm/tool_manipulator_description/urdf/tools/tool_3.xacro (robot description, xacro)
@@ -4,5 +4,7 @@
     <joint name="${prefix}tool_3_mount_joint" type="fixed"><parent link="${parent}"/><child link="${prefix}tool_3_link"/><origin xyz="0 0 0.015" rpy="${pi/2} 0 0"/></joint>
     <link name="${prefix}tool_3_link">
-      <visual><geometry><mesh filename="package://tool_manipulator_description/meshes/visual/long_phillipsbit.stl" scale="0.001 0.001 0.001"/></geometry><material name="motor_grey"/></visual>
+      <xacro:if value="${use_mesh}">
+        <visual><geometry><mesh filename="package://tool_manipulator_description/meshes/visual/long_phillipsbit.stl" scale="0.001 0.001 0.001"/></geometry><material name="motor_grey"/></visual>
+      </xacro:if>
       <collision><geometry><mesh filename="package://tool_manipulator_description/meshes/collision/long_phillipsbit.stl" scale="0.001 0.001 0.001"/></geometry></collision>
       <inertial><origin xyz="0 0.0283 0"/><mass value="0.050"/><inertia ixx="0.00002" ixy="0" ixz="0" iyy="0.000004" iyz="0" izz="0.00002"/></inertial>

Commit message: ㅈㅂ

File: src/arm/tool_manipulator_description/urdf/tool_manipulator.urdf.xacro (robot description, xacro)
@@ -203,10 +203,10 @@
     <origin xyz="-0.0184 0 0" rpy="0 -1.570796326795 0"/>
   </joint>
-  <!-- Former case 3 location: supply-box pickup area, not a measured grasp pose.
-       No permanent collision; reference axes are parallel to world. -->
+  <!-- Measured supply-box centre in arm_world/base_actuator. This is an object
+       reference point, not an executable TCP grasp pose. -->
   <link name="supplybox_pickup_area"/>
   <joint name="arm_world_to_supplybox_pickup_area" type="fixed">
     <parent link="arm_world"/><child link="supplybox_pickup_area"/>
-    <origin xyz="-0.268 -0.10245 0.153595589" rpy="0 0 0"/>
+    <origin xyz="-0.236197 -0.120 0.182" rpy="0 0 0"/>
   </joint>
   <!-- Former case 1 frame retained for its centre marker and dock references. -->
